File: kicad/mdb-esp32s3/mdb-esp32s3.kicad_sch (KiCad schematic)
At the start: 39 parts, among them J2 MDB_Connector, J3 Conn_02x09_Odd_Even, P1 USB_C_Plug_USB2.0, SW1 SW_Push, U1 ESP32-S3, U2 W25Q32JVSS, U4 LM317_SOT-223, U5 PC817, U6 PC817, Y1 Crystal

Commit message: refacting
Parts:
- removed C8: C, Capacitor_SMD:C_0603_1608Metric, symbol Device:C
- removed D2: LED, LED_SMD:LED_0603_1608Metric, symbol Device:LED
- removed R7: R, Resistor_SMD:R_0603_1608Metric, symbol Device:R
