File: kicad/mdb-esp32s3/mdb-esp32s3.kicad_pcb (KiCad board)
At the start: 2 copper layers, 42 x 47 mm, 36 parts, among them J2 MDB_Connector, J3 Conn_02x09_Odd_Even, P1 USB_C_Plug_USB2.0, SW1 SW_Push, U1 ESP32-S3, U2 W25Q32JVSS, U4 LM317_SOT-223, U5 PC817, U6 PC817, Y1 Crystal

Commit message: refacting
Parts:
- moved P1 0.45 mm to (96.5, 135.0)
Routing:
- net Net-(P1-CC): track 7.71 -> 9.11 mm
- net GND: track 194.0 -> 195.2 mm
- net Net-(D1-A): track 14.2 -> 15.2 mm

Commit message: refacting
Routing:
- net GND: track 195.2 -> 193.0 mm, vias 8 -> 7
- added copper zone on B.Cu, net GND
- added copper zone on F.Cu, net GND
