File: kicad/mdb-master-esp32s3/mdb-master-esp32s3.kicad_pcb (KiCad board)
At the start: 2 copper layers, 41.8 x 53.2 mm, 37 parts, among them J1 Conn_02x09_Odd_Even, J2 MDB_Connector, J3 Barrel_Jack, P1 USB_C_Plug_USB2.0, Q1 BC807, U2 LM317_SOT-223, Y1 Crystal

Commit message: Refacting
Parts:
- removed ESP32-S3FH4R2: ESP32-S3FH4R2, Package_DFN_QFN:QFN-56-1EP_7x7mm_P0.4mm_EP5.6x5.6mm
- added U1: ESP32-S3, Package_DFN_QFN:QFN-56-1EP_7x7mm_P0.4mm_EP5.6x5.6mm, F.Cu at (141.2, 117.7)
- moved C7 5.40 mm to (151.5, 132.8)
- moved D3 5.30 mm to (151.5, 138.0)
- moved C6 4.78 mm to (144.0, 127.0)
- moved R4 4.61 mm to (145.5, 109.0), turned to 90 degrees
- moved C4 4.52 mm to (144.0, 104.5)
- moved R1 4.50 mm to (139.3, 109.0)
- moved C5 4.50 mm to (139.3, 104.5)
- moved R15 4.28 mm to (157.1, 90.2), turned to 0 degrees
- moved R11 3.90 mm to (134.7, 136.0), turned to 180 degrees
- moved R10 3.15 mm to (134.7, 139.5), turned to 180 degrees
- moved Boot 0.28 mm to (127.0, 132.0)
- moved Reset 0.28 mm to (127.0, 138.2)
- moved R7 0.25 mm to (155.4, 131.2)
- moved R8 0.25 mm to (159.4, 131.2)
- moved J1 0.21 mm to (125.8, 105.8)
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Connections:
- J1 pad 11: /io6 -> unconnected-(J1-Pin_11-Pad11)
Routing:
- net GND: track 0.00 -> 217.4 mm, vias 0 -> 4
- net +3V3: track 0.00 -> 167.6 mm, vias 0 -> 11
- net +36V: track 0.00 -> 61.7 mm
- net /io5: track 0.00 -> 44.9 mm, vias 0 -> 2
- net Net-(U1-CHIP_PU/RESET): track 0.00 -> 40.8 mm, vias 0 -> 2
- net /io4: track 0.00 -> 40.4 mm, vias 0 -> 1
- net /boot: track 0.00 -> 38.2 mm, vias 0 -> 2
- net Net-(U1-LNA_IN/RF): track 0.00 -> 36.9 mm
- net /io21: track 0.00 -> 34.1 mm, vias 0 -> 2
- net /u0txd: track 0.00 -> 26.8 mm, vias 0 -> 1
- net /io6: track 0.00 -> 25.7 mm
- net /u0rxd: track 0.00 -> 24.4 mm, vias 0 -> 1
- net Net-(P1-SHIELD): track 0.00 -> 20.8 mm
- net Net-(U1-XTAL_P): track 0.00 -> 17.5 mm
- net Net-(U1-XTAL_N): track 0.00 -> 16.1 mm
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
Commit message: refacting
Routing:
- net GND: track 217.4 -> 220.5 mm
- net /io21: track 34.1 -> 32.6 mm
- added copper zone on F.Cu, net GND

Commit message: refacting
Parts:
- removed Boot: Boot, Button_Switch_SMD:SW_Tactile_SPST_NO_Straight_CK_PTS636Sx25SMTRLFS
- removed J1: Conn_02x09_Odd_Even, Connector_PinHeader_2.54mm:PinHeader_2x09_P2.54mm_Vertical
- removed Reset: Reset, Button_Switch_SMD:SW_Tactile_SPST_NO_Straight_CK_PTS636Sx25SMTRLFS
- added +3v3: TestPoint, TestPoint:TestPoint_Pad_D1.0mm, F.Cu at (152.4, 117.0)
- added J4: Conn_02x08_Odd_Even, Connector_PinHeader_2.54mm:PinHeader_2x08_P2.54mm_Vertical, F.Cu at (125.7, 109.2)
- added boot: Boot, Button_Switch_SMD:SW_Tactile_SPST_NO_Straight_CK_PTS636Sx25SMTRLFS, F.Cu at (126.9, 132.4)
- added gnd: TestPoint, TestPoint:TestPoint_Pad_D1.0mm, F.Cu at (148.8, 118.4)
- added reset: Reset, Button_Switch_SMD:SW_Tactile_SPST_NO_Straight_CK_PTS636Sx25SMTRLFS, F.Cu at (126.9, 138.4)
- added vin: TestPoint, TestPoint:TestPoint_Pad_D1.0mm, F.Cu at (162.4, 129.4)
- moved U2 12.5 mm to (158.6, 124.3)
- moved J3 12.2 mm to (153.4, 135.8)
- moved R8 11.5 mm to (152.4, 122.1), turned to -90 degrees
- moved BZ1 8.21 mm to (128.2, 103.4), turned to 90 degrees
- moved C1 8.21 mm to (136.6, 101.6), turned to 180 degrees
- moved C7 7.68 mm to (148.8, 125.6)
- moved R15 6.81 mm to (153.8, 96.2), turned to 90 degrees
- moved R7 5.66 mm to (152.4, 126.4), turned to -90 degrees
- moved L1 4.68 mm to (136.6, 99.6)
- moved AE1 4.63 mm to (138.2, 98.0)
- moved C6 4.01 mm to (140.2, 128.2)
- moved Y1 3.64 mm to (142.1, 101.8)
- moved C4 3.03 mm to (145.0, 107.3)
- moved C5 2.98 mm to (140.2, 107.3)
- moved U1 2.96 mm to (139.3, 119.9)
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Connections:
- net +36V renamed /vin
Routing:
- net GND: track 220.5 -> 0.00 mm, vias 4 -> 0
- net +3V3: track 167.8 -> 0.00 mm, vias 11 -> 0
- net /vin: track 61.7 -> 0.00 mm
- net /io5: track 44.9 -> 0.00 mm, vias 2 -> 0
- net Net-(U1-CHIP_PU/RESET): track 40.8 -> 0.00 mm, vias 2 -> 0
- net /io4: track 40.4 -> 0.00 mm, vias 1 -> 0
- net /boot: track 38.2 -> 0.00 mm, vias 2 -> 0
- net Net-(U1-LNA_IN/RF): track 36.9 -> 0.00 mm
- net /io21: track 32.6 -> 0.00 mm, vias 2 -> 0
- net /u0txd: track 26.8 -> 0.00 mm, vias 1 -> 0
- net /io6: track 25.7 -> 0.00 mm
- net /u0rxd: track 24.4 -> 0.00 mm, vias 1 -> 0
- net Net-(P1-SHIELD): track 20.8 -> 0.00 mm
- net Net-(U1-XTAL_P): track 17.5 -> 0.00 mm
- net Net-(U1-XTAL_N): track 16.1 -> 0.00 mm
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- removed copper zone on F.Cu, net GND
Other:
- board size 41.8 x 53.2 mm -> 41.8 x 48.7 mm

Commit message: Refacting
Parts:
- moved +3v3 4.47 mm to (148.4, 119.0)
- moved gnd 4.29 mm to (152.6, 116.4)
- moved vin 0.72 mm to (161.8, 129.8)
- moved reset 0.08 mm to (127.0, 138.4)

Commit message: Refacting
Parts:
- removed J4: Conn_02x08_Odd_Even, Connector_PinHeader_2.54mm:PinHeader_2x08_P2.54mm_Vertical
- removed boot: Boot, Button_Switch_SMD:SW_Tactile_SPST_NO_Straight_CK_PTS636Sx25SMTRLFS
- removed reset: Reset, Button_Switch_SMD:SW_Tactile_SPST_NO_Straight_CK_PTS636Sx25SMTRLFS
- added B: Boot, Button_Switch_SMD:SW_Tactile_SPST_NO_Straight_CK_PTS636Sx25SMTRLFS, F.Cu at (127.1, 133.5)
- added J5: Conn_02x10_Odd_Even, Connector_PinHeader_2.54mm:PinHeader_2x10_P2.54mm_Vertical, F.Cu at (125.8, 105.6)
- added R: Reset, Button_Switch_SMD:SW_Tactile_SPST_NO_Straight_CK_PTS636Sx25SMTRLFS, F.Cu at (127.1, 138.5)
- moved +3v3 26.5 mm to (153.5, 93.0)
- moved gnd 16.1 mm to (162.0, 129.5)
- moved vin 15.8 mm to (152.5, 117.0)
- moved BZ1 7.60 mm to (132.3, 97.0), turned to 180 degrees
- moved AE1 1.57 mm to (138.9, 96.6)
- moved C1 1.10 mm to (136.6, 100.5)
- moved L1 1.10 mm to (136.6, 98.5)
- moved R4 0.88 mm to (144.3, 110.6)
- moved C7 0.70 mm to (149.5, 125.5), turned to -90 degrees
- moved C5 0.41 mm to (139.8, 107.3)
- moved C6 0.41 mm to (139.8, 128.2), turned to 180 degrees
- moved R1 0.41 mm to (139.8, 110.6), turned to 180 degrees
- turned C3 to 180 degrees
Routing:
- net GND: track 0.00 -> 217.3 mm, vias 0 -> 5
- net +3V3: track 0.00 -> 135.4 mm, vias 0 -> 7
- net /vin: track 0.00 -> 75.5 mm, vias 0 -> 2
- net /io4: track 0.00 -> 65.3 mm, vias 0 -> 1
- net /io5: track 0.00 -> 59.7 mm, vias 0 -> 3
- net /boot: track 0.00 -> 49.6 mm, vias 0 -> 2
- net Net-(U1-CHIP_PU/RESET): track 0.00 -> 47.9 mm, vias 0 -> 2
- net /io21: track 0.00 -> 33.4 mm, vias 0 -> 2
- net /u0txd: track 0.00 -> 26.7 mm, vias 0 -> 1
- net /u0rxd: track 0.00 -> 26.5 mm, vias 0 -> 1
- net /io6: track 0.00 -> 23.7 mm
- net Net-(P1-SHIELD): track 0.00 -> 20.4 mm
- net Net-(U1-LNA_IN/RF): track 0.00 -> 18.5 mm
- net Net-(U1-XTAL_N): track 0.00 -> 18.2 mm
- net Net-(U1-XTAL_P): track 0.00 -> 16.7 mm
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- added copper zone on F.Cu, net GND
Other:
- board size 41.8 x 48.7 mm -> 41.8 x 50.2 mm

Commit message: refacting
Parts:
- moved gnd 16.4 mm to (145.8, 126.9)
- moved +3v3 7.79 mm to (161.3, 93.1)
- moved vin 0.99 mm to (151.5, 117.1)
Routing:
- net GND: track 217.3 -> 230.0 mm
- net +3V3: track 135.4 -> 133.0 mm, vias 7 -> 8
- net /vin: track 75.5 -> 76.4 mm, vias 2 -> 0

Commit message: Refacting pcb
Parts:
- renumbered U1 to ESP32-S3
Routing:
- net +3V3: track 133.0 -> 133.5 mm
Changed lines of the file:
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@@
 		(tags "capacitor")
 		(property "Reference" "C2"
-			(at 0.1 2 180)
+			(at 0.007 1.708 180)
 			(layer "F.SilkS")
 			(effects
@@
 		(descr "QFN, 56 Pin (http://www.cypress.com/file/416486/download#page=40), generated with kicad-footprint-generator ipc_noLead_generator.py")
 		(tags "QFN NoLead")
-		(property "Reference" "U1"
+		(property "Reference" "ESP32-S3"
 			(at 0 -4.83 135)
 			(layer "F.SilkS")
@@
 		)
 		(property "Value" "ESP32-S3"
-			(at 0 4.83 135)
+			(at -0.761797 -5.046157 135)
 			(layer "F.Fab")
+			(hide yes)
 			(effects
 				(font
@@
 		(tags "resistor")
 		(property "Reference" "R8"
-			(at 0 1.5 90)
+			(at -0.693 1.5 90)
 			(layer "F.SilkS")
 			(effects
@@
 	)
 	(segment
-		(start 149.5 113.8)
-		(end 149.5 118.004)
+		(start 149.5 118.004)
+		(end 152.076 120.58)
 		(width 0.2)
 		(layer "F.Cu")
@@
 	)
 	(segment
-		(start 124.7 104.49)
-		(end 125.85 105.64)
+		(start 152.662648 122.23)
+		(end 151.937352 122.23)
 		(width 0.2)
 		(layer "F.Cu")
@@
 	)
 	(segment
-		(start 156.0375 118.6)
-		(end 159.4 121.9625)
+		(start 124.7 104.49)
+		(end 125.85 105.64)
 		(width 0.2)
 		(layer "F.Cu")
@@
 	)
 	(segment
-		(start 153.289 121.603648)
-		(end 152.662648 122.23)
+		(start 156.0375 118.6)
+		(end 159.4 121.9625)
 		(width 0.2)
 		(layer "F.Cu")
@@
 	)
 	(segment
-		(start 149.5 118.004)
-		(end 152.076 120.58)
+		(start 151.13 123.037352)
+		(end 151.13 125.22)
 		(width 0.2)
 		(layer "F.Cu")
@@
 	)
 	(segment
-		(start 152.076 120.58)
-		(end 152.912648 120.58)
+		(start 135.8125 98.5)
+		(end 135.8125 98.6875)
 		(width 0.2)
 		(layer "F.Cu")
@@
 	)
 	(segment
-		(start 135.8125 98.5)
-		(end 135.8125 98.6875)
+		(start 133.675 139.5)
+		(end 133.675 136)
 		(width 0.2)
 		(layer "F.Cu")
@@
 	)
 	(segment
-		(start 133.675 139.5)
-		(end 133.675 136)
+		(start 153.289 121.603648)
+		(end 152.662648 122.23)
 		(width 0.2)
 		(layer "F.Cu")
@@
 	)
 	(segment
-		(start 151.13 123.037352)
-		(end 151.13 125.22)
-		(width 0.2)
-		(layer "F.Cu")
-		(net 3)
-	)
-	(segment
 		(start 124.7 97)
 		(end 124.7 104.49)
@@
 	)
 	(segment
-		(start 153.289 120.956352)
-		(end 153.289 121.603648)
+		(start 152.912648 120.58)
+		(end 153.289 120.956352)
 		(width 0.2)
 		(layer "F.Cu")
@@
 	)
 	(segment
-		(start 152.662648 122.23)
-		(end 151.937352 122.23)
+		(start 149.477 126.873)
+		(end 149.5 126.85)
 		(width 0.2)
 		(layer "F.Cu")
@@
 	)
 	(segment
-		(start 149.477 126.873)
-		(end 149.5 126.85)
+		(start 153.289 120.956352)
+		(end 153.289 121.603648)
 		(width 0.2)
 		(layer "F.Cu")
@@
 	)
 	(segment
+		(start 149.5 113.8)
+		(end 149.5 118.004)
+		(width 0.2)
+		(layer "F.Cu")
+		(net 3)
+	)
+	(segment
 		(start 142.75 100.75)
 		(end 144.25 102.25)
@@
 	)
 	(segment
+		(start 151.13 125.22)
+		(end 149.5 126.85)
+		(width 0.2)
+		(layer "F.Cu")
+		(net 3)
+	)
+	(segment
 		(start 136.575 100.923696)
 		(end 136.926304 101.275)
@@
 	)
 	(segment
-		(start 151.937352 122.23)
-		(end 151.13 123.037352)
+		(start 140.5375 128.2)
+		(end 141.95 128.2)
 		(width 0.2)
 		(layer "F.Cu")
@@
 	)
 	(segment
-		(start 140.5375 128.2)
-		(end 141.95 128.2)
+		(start 152.076 120.58)
+		(end 152.912648 120.58)
 		(width 0.2)
 		(layer "F.Cu")
@@
 	)
 	(segment
-		(start 151.13 125.22)
-		(end 149.5 126.85)
+		(start 151.937352 122.23)
+		(end 151.13 123.037352)
 		(width 0.2)
 		(layer "F.Cu")
@@
 	)
 	(segment
-		(start 152.912648 120.58)
-		(end 153.289 120.956352)
-		(width 0.2)
-		(layer "F.Cu")
-		(net 3)
-	)
-	(segment
 		(start 149.35 137.85)
 		(end 157.35 137.85)
@@
 	)
 	(segment
-		(start 156.225 96.676948)
-		(end 159.810948 93.091)
+		(start 147.32 114)
+		(end 147.248242 114)
 		(width 0.2)
 		(layer "F.Cu")
@@
 	)
 	(segment
-		(start 150.2 111.087648)
-		(end 147.95 113.337648)
+		(start 156.225 96.676948)
+		(end 159.810948 93.091)
 		(width 0.2)
 		(layer "F.Cu")
@@
 	)
 	(segment
-		(start 156.225 97.13)
-		(end 156.225 96.676948)
-		(width 0.2)
-		(layer "F.Cu")
-		(net 5)
-	)
-	(segment
-		(start 154.883452 104.15)
-		(end 153.35 104.15)
+		(start 147.95 113.337648)
+		(end 147.95 113.8)
 		(width 0.2)
 		(layer "F.Cu")
@@
 	)
 	(segment
-		(start 156.75 97.655)
-		(end 156.75 102.283452)
+		(start 156.225 97.13)
+		(end 156.225 96.676948)
 		(width 0.2)
 		(layer "F.Cu")
@@
 	)
 	(segment
-		(start 155.45 124.645406)
-		(end 155.45 124.3)
+		(start 156.75 102.283452)
+		(end 154.883452 104.15)
 		(width 0.2)
 		(layer "F.Cu")
@@
 	)
 	(segment
-		(start 150.459 124.15)
-		(end 150.53 124.079)
+		(start 156.75 97.655)
+		(end 156.75 102.283452)
 		(width 0.2)
 		(layer "F.Cu")
@@
 	)
 	(segment
-		(start 147.95 113.337648)
-		(end 147.95 113.8)
+		(start 150.2 107.3)
+		(end 150.2 111.087648)
 		(width 0.2)
 		(layer "F.Cu")
@@
 	)
 	(segment
-		(start 143.0375 124.15)
-		(end 149.5 124.15)
+		(start 155.45 124.645406)
+		(end 155.45 124.3)
 		(width 0.2)
 		(layer "F.Cu")
@@
 	)
 	(segment
-		(start 149.5 123.8175)
-		(end 152.0375 121.28)
+		(start 147.95 118.232)
+		(end 147.95 113.8)
 		(width 0.2)
 		(layer "F.Cu")
@@
 	)
 	(segment
-		(start 138.462455 115.944529)
-		(end 138.084959 115.567035)
+		(start 150.459 124.15)
+		(end 150.53 124.079)
 		(width 0.2)
 		(layer "F.Cu")
@@
 	)
 	(segment
-		(start 156.75 102.283452)
-		(end 154.883452 104.15)
+		(start 143.0375 124.15)
+		(end 149.5 124.15)
 		(width 0.2)
 		(layer "F.Cu")
@@
 	)
 	(segment
-		(start 138.179613 116.227371)
-		(end 138.462455 115.944529)
+		(start 149.5 123.8175)
+		(end 152.0375 121.28)
 		(width 0.2)
 		(layer "F.Cu")
@@
 	)
 	(segment
-		(start 155.45 124.3)
-		(end 155.445 124.3)
+		(start 147.248242 114)
+		(end 142.758129 118.490113)
 		(width 0.2)
 		(layer "F.Cu")
@@
 	)
 	(segment
-		(start 135.325 110.6)
-		(end 135.325 107.35)
+		(start 147.32 114)
+		(end 147.75 114)
 		(width 0.2)
 		(layer "F.Cu")
@@
 	)
 	(segment
-		(start 150.2 107.3)
-		(end 150.2 111.087648)
+		(start 138.462455 115.944529)
+		(end 138.084959 115.567035)
 		(width 0.2)
 		(layer "F.Cu")
@@
 	)
 	(segment
-		(start 139.929702 115.661686)
-		(end 140.212543 115.944527)
+		(start 138.179613 116.227371)
+		(end 138.462455 115.944529)
 		(width 0.2)
 		(layer "F.Cu")
@@
 	)
 	(segment
-		(start 147.75 114)
-		(end 147.95 113.8)
+		(start 155.45 124.3)
+		(end 155.445 124.3)
 		(width 0.2)
 		(layer "F.Cu")
@@
 	)
 	(segment
-		(start 156.225 97.13)
-		(end 156.75 97.655)
+		(start 135.325 110.6)
+		(end 135.325 107.35)
+		(width 0.2)
+		(layer "F.Cu")
+		(net 5)
+	)
+	(segment
+		(start 139.929702 115.661686)
+		(end 140.212543 115.944527)
 		(width 0.2)
 		(layer "F.Cu")
@@
 	)
 	(segment
-		(start 146.177 115.071242)
-		(end 142.758129 118.490113)
+		(start 152.425 121.28)
+		(end 150.998 121.28)
 		(width 0.2)
 		(layer "F.Cu")
@@
 	)
 	(segment
-		(start 146.177 114)
-		(end 147.75 114)
+		(start 156.225 97.13)
+		(end 156.75 97.655)
 		(width 0.2)
 		(layer "F.Cu")
@@
 	)
 	(segment
-		(start 152.425 121.28)
-		(end 150.998 121.28)
+		(start 161.975 124.075)
+		(end 161.75 124.3)
 		(width 0.2)
 		(layer "F.Cu")
@@
 	)
 	(segment
-		(start 161.975 124.075)
-		(end 161.75 124.3)
+		(start 154.883452 104.15)
+		(end 153.35 104.15)
 		(width 0.2)
 		(layer "F.Cu")
@@
 	)
 	(segment
-		(start 146.177 114)
-		(end 146.177 115.071242)
+		(start 152.0375 121.28)
+		(end 152.425 121.28)
 		(width 0.2)
 		(layer "F.Cu")
@@
 	)
 	(segment
-		(start 152.0375 121.28)
-		(end 152.425 121.28)
+		(start 150.2 111.087648)
+		(end 147.95 113.337648)
 		(width 0.2)
 		(layer "F.Cu")
@@
 	)
 	(segment
-		(start 147.95 118.232)
+		(start 147.75 114)
 		(end 147.95 113.8)
 		(width 0.2)
@@
 	)
 	(via
-		(at 146.177 114)
+		(at 147.32 114)
 		(size 0.6)
 		(drill 0.3)
@@
 	)
 	(segment
-		(start 144.4 114)
-		(end 141.9 111.5)
+		(start 147.32 114)
+		(end 144.4 114)
 		(width 0.2)
 		(layer "B.Cu")
@@
 	)
 	(segment
+		(start 144.4 114)
+		(end 141.9 111.5)
+		(width 0.2)
+		(layer "B.Cu")
+		(net 5)
+	)
+	(segment
 		(start 150.751 124.3)
 		(end 155.45 124.3)
@@
 		(width 0.2)
 		(layer "B.Cu")
-		(net 5)
-	)
-	(segment
-		(start 146.177 114)
-		(end 144.4 114)
-		(width 0.2)
-		(layer "B.Cu")

Commit message: refacting
Other:
- board text added: "7 gnd 8 gnd 9 tx 10 rx 11 1 12 2 13 4 14 5 +3v3 17 vin 18"
Changed lines of the file:
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@@
 			(outputformat 1)
 			(mirror no)
-			(drillshape 1)
+			(drillshape 0)
 			(scaleselection 1)
-			(outputdirectory "")
+			(outputdirectory "../../../../Downloads/mdb-master/")
 		)
 	)
@@
 		(layer "Edge.Cuts")
 	)
+	(gr_text "7		gnd\n8		gnd\n9		tx\n10		rx	\n11		1\n12		2\n13		4\n14		5\n+3v3	17\nvin		18"
+		(at 142.875 124.587 0)
+		(layer "B.SilkS")
+		(effects
+			(font
+				(size 1 1)
+				(thickness 0.1)
+			)
+			(justify left bottom mirror)
+		)
+	)
 	(segment
