File: kicad/mdb-master-esp32s3/mdb-master-esp32s3.kicad_pcb (KiCad board)
At the start: 2 copper layers, 41 x 46 mm, 33 parts, among them J1 MDB_Connector, J2 Barrel_Jack, J3 USB_C_Receptacle_USB2.0_16P, J4 Conn_02x11_Odd_Even, Q1 BC807, SW1 SW_Push, U1 ESP32-S3R8, U2 AMS1117-3.3, Y1 40000hz

Commit message: Refacting kicad
Other:
- board text added: "mdb-master-esp32s3"
Changed lines of the file:
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@@
 		(layer "Edge.Cuts")
 	)
+	(gr_text "mdb-master-esp32s3"
+		(at 144 78 0)
+		(layer "B.SilkS")
+		(effects
+			(font
+				(size 1 1)
+				(thickness 0.1)
+			)
+			(justify left bottom mirror)
+		)
+	)
 	(gr_text "10"
 		(at 134.4346 91.661 0)
@@
 	)
 	(segment
-		(start 147.89184 112.449809)
-		(end 147.9848 112.542769)
+		(start 153.525 100.225)
+		(end 153.75 100.225)
 		(width 0.5)
 		(layer "F.Cu")
@@
 	)
 	(segment
-		(start 153.025 100.225)
-		(end 153 100.25)
+		(start 147.89184 112.449809)
+		(end 147.9848 112.542769)
 		(width 0.5)
 		(layer "F.Cu")
@@
 	)
 	(segment
-		(start 153.75 100.225)
-		(end 153.025 100.225)
-		(width 0.5)
-		(layer "F.Cu")
-		(net 3)
-	)
-	(segment
 		(start 141.5848 113.82)
 		(end 141.0648 113.82)
@@
 	)
 	(segment
+		(start 145.25 96.3625)
+		(end 143.2375 94.35)
+		(width 0.2)
+		(layer "F.Cu")
+		(net 3)
+	)
+	(segment
 		(start 137.1664 119.7414)
 		(end 135 117.575)
@@
 	)
 	(segment
-		(start 158.55 96.312352)
-		(end 158.887352 95.975)
-		(width 0.2)
+		(start 153 100.75)
+		(end 153.525 100.225)
+		(width 0.5)
 		(layer "F.Cu")
 		(net 3)
 	)
 	(segment
-		(start 145.25 96.3625)
-		(end 143.2375 94.35)
+		(start 158.55 96.312352)
+		(end 158.887352 95.975)
 		(width 0.2)
 		(layer "F.Cu")
@@
 	)
 	(via
-		(at 153 100.25)
+		(at 153 100.75)
 		(size 0.6)
 		(drill 0.3)
@@
 	)
 	(segment
-		(start 147.045461 111.5)
-		(end 147.89184 112.346379)
+		(start 153 100.75)
+		(end 148.744157 105.005843)
 		(width 0.5)
 		(layer "B.Cu")
@@
 	)
 	(segment
-		(start 147.89184 112.346379)
-		(end 147.89184 112.449809)
+		(start 147.045461 111.5)
+		(end 147.89184 112.346379)
 		(width 0.5)
 		(layer "B.Cu")
@@
 	)
 	(segment
-		(start 148.744157 105.005843)
-		(end 146.817202 105.005843)
+		(start 147.89184 112.346379)
+		(end 147.89184 112.449809)
 		(width 0.5)
 		(layer "B.Cu")
@@
 	)
 	(segment
-		(start 140.75 111.5)
-		(end 142.912164 111.5)
-		(width 0.5)
-		(layer "B.Cu")
-		(net 3)
-	)
-	(segment
-		(start 142.912164 111.5)
-		(end 147.045461 111.5)
+		(start 148.744157 105.005843)
+		(end 146.817202 105.005843)
 		(width 0.5)
 		(layer "B.Cu")
@@
 	)
 	(segment
-		(start 153 100.75)
-		(end 148.744157 105.005843)
+		(start 140.75 111.5)
+		(end 142.912164 111.5)
 		(width 0.5)
 		(layer "B.Cu")
@@
 	)
 	(segment
-		(start 153 100.25)
-		(end 153 100.75)
+		(start 142.912164 111.5)
+		(end 147.045461 111.5)
 		(width 0.5)
 		(layer "B.Cu")
@@
 	)
 	(segment
-		(start 147.11573 108.13427)
-		(end 149.945629 105.304371)
-		(width 0.2)
-		(layer "F.Cu")
-		(net 5)
-	)
-	(segment
 		(start 143.25 96.7375)
 		(end 143.2375 96.75)
@@
 	)
 	(segment
-		(start 149.945629 105.304371)
-		(end 149.945629 104.245183)
-		(width 0.2)
-		(layer "F.Cu")
-		(net 5)
-	)
-	(segment
 		(start 158.55 103.75)
 		(end 160 102.3)
@@
 	)
 	(segment
-		(start 149.850223 104.149777)
-		(end 147.350106 101.64966)
+		(start 149.945629 104.445629)
+		(end 149.625 104.125)
 		(width 0.2)
 		(layer "F.Cu")
@@
 	)
 	(segment
+		(start 147.11573 108.13427)
+		(end 149.945629 105.304371)
+		(width 0.2)
+		(layer "F.Cu")
+		(net 5)
+	)
+	(segment
 		(start 147.225 98.25)
 		(end 147.225 99)
@@
 	)
 	(segment
-		(start 153.75 101.775)
-		(end 152.027944 101.775)
+		(start 149.625 104.125)
+		(end 147.350106 101.850106)
 		(width 0.2)
 		(layer "F.Cu")
@@
 	)
 	(segment
-		(start 144.920118 106.670118)
-		(end 146.38427 108.13427)
+		(start 153.75 101.775)
+		(end 152.027944 101.775)
 		(width 0.2)
 		(layer "F.Cu")
@@
 	)
 	(segment
-		(start 147.350106 101.361669)
-		(end 147.701085 101.01069)
-		(width 0.2)
-		(layer "F.Cu")
-		(net 5)
-	)
-	(segment
-		(start 149.850223 103.952721)
-		(end 149.850223 104.149777)
+		(start 149.677944 104.125)
+		(end 149.625 104.125)
 		(width 0.2)
 		(layer "F.Cu")
@@
 	)
 	(segment
-		(start 144.304398 106.670118)
-		(end 144.920118 106.670118)
+		(start 142.136196 93.575)
+		(end 142.4375 93.876304)
 		(width 0.2)
 		(layer "F.Cu")
@@
 	)
 	(segment
-		(start 142.136196 93.575)
-		(end 142.4375 93.876304)
+		(start 141.21875 109.5)
+		(end 141.474517 109.5)
 		(width 0.2)
 		(layer "F.Cu")
@@
 	)
 	(segment
-		(start 141.21875 109.5)
-		(end 141.474517 109.5)
+		(start 144.920118 106.670118)
+		(end 146.38427 108.13427)
 		(width 0.2)
 		(layer "F.Cu")
@@
 	)
 	(segment
-		(start 149.945629 104.245183)
-		(end 149.850223 104.149777)
+		(start 144.304398 106.670118)
+		(end 144.920118 106.670118)
 		(width 0.2)
 		(layer "F.Cu")
@@
 	)
 	(segment
-		(start 147.350106 101.64966)
-		(end 147.350106 101.361669)
+		(start 147.350106 101.361669)
+		(end 147.701085 101.01069)
 		(width 0.2)
 		(layer "F.Cu")
@@
 	)
 	(segment
+		(start 143.95342 107.021097)
+		(end 144.304398 106.670118)
+		(width 0.2)
+		(layer "F.Cu")
+		(net 5)
+	)
+	(segment
 		(start 147.225 99)
 		(end 147.225 100.534605)
@@
 	(segment
 		(start 150.24667 103.556274)
-		(end 149.850223 103.952721)
+		(end 149.677944 104.125)
+		(width 0.2)
+		(layer "F.Cu")
+		(net 5)
+	)
+	(segment
+		(start 149.945629 105.304371)
+		(end 149.945629 104.445629)
 		(width 0.2)
 		(layer "F.Cu")
@@
 	)
 	(segment
+		(start 147.350106 101.850106)
+		(end 147.350106 101.361669)
+		(width 0.2)
+		(layer "F.Cu")
+		(net 5)
+	)
+	(segment
 		(start 160 102.3)
 		(end 160 97.45)
@@
 		(net 5)
 	)
-	(segment
-		(start 143.95342 107.021097)
-		(end 144.304398 106.670118)
-		(width 0.2)
-		(layer "F.Cu")
-		(net 5)
-	)
 	(via
 		(at 142.625 96.125)
@@
 	)
 	(segment
-		(start 145.75 110.25)
-		(end 145.35858 109.85858)
+		(start 129.8696 111.4)
+		(end 131.5396 113.07)
 		(width 0.2)
 		(layer "B.Cu")
@@
 	)
 	(segment
-		(start 129.8696 111.4)
-		(end 131.5396 113.07)
+		(start 148.120178 113.07)
+		(end 148.5 112.690178)
 		(width 0.2)
 		(layer "B.Cu")
@@
 	)
 	(segment
-		(start 148.5 112.690178)
-		(end 148.5 112.176721)
+		(start 146 110.5)
+		(end 145.35858 109.85858)
 		(width 0.2)
 		(layer "B.Cu")
@@
 	)
 	(segment
-		(start 131.5396 113.07)
-		(end 148.120178 113.07)
+		(start 148.5 112.690178)
+		(end 148.5 112.176721)
 		(width 0.2)
 		(layer "B.Cu")
@@
 	)
 	(segment
-		(start 146.573279 110.25)
-		(end 145.75 110.25)
+		(start 131.5396 113.07)
+		(end 148.120178 113.07)
 		(width 0.2)
 		(layer "B.Cu")
@@
 	)
 	(segment
-		(start 148.120178 113.07)
-		(end 148.5 112.690178)
+		(start 146.823279 110.5)
+		(end 146 110.5)
 		(width 0.2)
 		(layer "B.Cu")
@@
 	(segment
 		(start 148.5 112.176721)
-		(end 146.573279 110.25)
+		(end 146.823279 110.5)
 		(width 0.2)
 		(layer "B.Cu")
@@
 	)
 	(segment
-		(start 153.6 94.35)
-		(end 150.375 97.575)
+		(start 152.25 98.158832)
+		(end 148.549614 101.859218)
 		(width 0.2)
 		(layer "F.Cu")
@@
 	)
 	(segment
-		(start 150.375 100.033832)
-		(end 148.549614 101.859218)
+		(start 153.6 94.35)
+		(end 152.25 95.7)
 		(width 0.2)
 		(layer "F.Cu")
@@
 	)
 	(segment
-		(start 150.375 97.575)
-		(end 150.375 100.033832)
+		(start 152.25 95.7)
+		(end 152.25 98.158832)
 		(width 0.2)
 		(layer "F.Cu")
@@
 	)
 	(segment
+		(start 141.6875 96.7375)
+		(end 141.675 96.75)
+		(width 0.2)
+		(layer "F.Cu")
+		(net 65)
+	)
+	(segment
 		(start 141.675 96.752371)
 		(end 145.933319 101.01069)
@@
 		(start 141.6875 94.35)
 		(end 141.6875 96.7375)
-		(width 0.5)
+		(width 0.2)
 		(layer "F.Cu")
 		(net 65)
@@
 		(layer "F.Cu")
 		(net 65)
-	)
-	(segment
-		(start 141.6875 96.7375)
-		(end 141.675 96.75)
-		(width 0.5)
-		(layer "F.Cu")
-		(net 65)

Commit message: Master initial routing
Parts:
- removed AE1: Antenna, RF_Antenna:Texas_SWRA117D_2.4GHz_Left
- removed C1: 0.1uF, Capacitor_SMD:C_0603_1608Metric
- removed C2: 1uF, Capacitor_SMD:C_0603_1608Metric
- removed L1: 2nH, Inductor_SMD:L_0603_1608Metric
- removed R10, R11: 240ohm, Resistor_SMD:R_0603_1608Metric
- added C10: 0.1uF, Capacitor_SMD:C_0603_1608Metric, F.Cu at (171.2, 123.5)
- added C11: 0.1uF, Capacitor_SMD:C_0603_1608Metric, F.Cu at (172.0, 92.1)
- added C12: 100uF, Capacitor_SMD:CP_Elec_6.3x5.8, F.Cu at (160.3, 108.0)
- added C13: 220uF, Capacitor_Tantalum_SMD:CP_EIA-3528-21_Kemet-B, F.Cu at (151.8, 108.6)
- added C8: 1uF, Capacitor_SMD:C_0603_1608Metric, F.Cu at (171.2, 112.7)
- added C9: 0.1uF, Capacitor_SMD:C_0603_1608Metric, F.Cu at (171.9, 117.6)
- added FB1: FerriteBead_Small, Inductor_SMD:L_0603_1608Metric, F.Cu at (143.1, 93.0)
- added TP1: TestPoint, TestPoint:TestPoint_Pad_D1.0mm, F.Cu at (180.9, 117.1)
- added TP2: TestPoint, TestPoint:TestPoint_Pad_D1.0mm, F.Cu at (180.9, 120.1)
- C3: value 10uF -> 1uF
- C4: value 1.8pf -> 12pF
- C5: value 22pf -> 12pF
- C6: value 22pf -> 10uF
- C7: value 1uF -> 0.1uF
- D1: value 1N5819HWQ -> XL-2121RGBC-2812B; footprint Diode_SMD:D_SOD-123 -> LED_SMD:LED_WS2812B-2020_PLCC4_2.0x2.0mm
- D2, D3: value LED -> D_Schottky; footprint LED_SMD:LED_0603_1608Metric -> Diode_SMD:D_SOD-123
- J1: value MDB_Connector -> Conn_02x11_Odd_Even; footprint Connector_Molex:Molex_Mini-Fit_Jr_5566-06A_2x03_P4.20mm_Vertical -> Connector_PinHeader_2.54mm:PinHeader_2x11_P2.54mm_Vertical
- J2: value Barrel_Jack -> USB_C_Receptacle_USB2.0_16P; footprint Connector_BarrelJack:BarrelJack_Horizontal -> Connector_USB:USB_C_Receptacle_G-Switch_GT-USB-7010ASV
- J3: value USB_C_Receptacle_USB2.0_16P -> MDB_Connector; footprint Connector_USB:USB_C_Receptacle_G-Switch_GT-USB-7010ASV -> Connector_Molex:Molex_Mini-Fit_Jr_5566-06A_2x03_P4.20mm_Vertical
- J4: value Conn_02x11_Odd_Even -> Barrel_Jack; footprint Connector_PinHeader_2.54mm:PinHeader_2x11_P2.54mm_Vertical -> Connector_BarrelJack:BarrelJack_Horizontal
- L2: value 2.4nh -> 100uH; footprint Inductor_SMD:L_0603_1608Metric -> Inductor_SMD:L_7.3x7.3_H3.5
- R1, R3, R4: value 3.3k -> 10k
- R2: value 180ohm -> 10k
- R5, R6: value 3.3k -> 5.1k
- R7, R9: value 3.3k -> 1k
- R8: value 3.3k -> 4k7
- U1: value ESP32-S3R8 -> ESP32-S3FH4R2
- U2: value AMS1117-3.3 -> LM2594HVM-3.3; footprint Package_TO_SOT_SMD:SOT-223 -> Package_SO:SOIC-8_3.9x4.9mm_P1.27mm
- Y1: value 40000hz -> Crystal_GND24; footprint Crystal:Crystal_HC49-4H_Vertical -> Crystal:Crystal_SMD_3225-4Pin_3.2x2.5mm
- moved R8 55.5 mm to (134.0, 63.6)
- moved R9 55.5 mm to (134.0, 59.2)
- moved R7 48.1 mm to (120.3, 60.4)
- moved R5 38.8 mm to (136.9, 117.8), turned to -90 degrees
- moved J3 38.4 mm to (140.5, 79.3)
- moved L2 36.4 mm to (152.8, 116.6)
- moved J1 34.0 mm to (130.0, 86.0), turned to 0 degrees
- moved D1 32.4 mm to (174.9, 92.2), turned to 0 degrees
- moved Q1 27.1 mm to (126.9, 60.7)
- moved J4 25.9 mm to (155.5, 82.7), turned to 180 degrees
- moved R6 25.0 mm to (136.5, 114.2), turned to 90 degrees
- moved R1 23.8 mm to (173.9, 69.2)
- moved D2 23.2 mm to (146.4, 109.8)
- moved C4 21.2 mm to (158.3, 92.4), turned to 90 degrees
- moved R2 17.7 mm to (152.6, 97.0), turned to 0 degrees
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Connections:
- C3 pad 1: GND -> /reset
- C3 pad 2: +3V3 -> GND
- C4 pad 1: Net-(AE1-A) -> GND
- C4 pad 2: Net-(U1-LNA_IN/RF) -> Net-(U1-XTAL_N)
- C5 pad 2: Net-(U1-XTAL_N) -> Net-(U1-XTAL_P)
- C6 pad 2: Net-(U1-XTAL_P) -> +3V3
- D1 pad 1: /vin -> unconnected-(D1-DOUT-Pad1)
- D1 pad 2: Net-(D1-A) -> GND
- D2 pad 1: GND -> /vin
- D3 pad 1: GND -> Net-(D3-K)
- D3 pad 2: Net-(D3-A) -> GND
- J1 pad 1: /vin -> /u0txd
- J1 pad 2: GND -> /reset
- J1 pad 3: unconnected-(J1-Pin_3-Pad3) -> /u0rxd
- J1 pad 4: /io4 -> /io8
- J1 pad 5: /mdb_master_transmit -> /io1
- J1 pad 6: GND -> /io9
- J4 pad 1: /u0txd -> /vin
- J4 pad 2: /io8 -> GND
- J4 pad 3: /u0rxd -> (no net)
- L2 pad 1: GND -> Net-(D3-K)
- L2 pad 2: Net-(AE1-A) -> +3V3
- R1 pad 2: /io4 -> /reset
- R2 pad 1: /mdb_master_transmit -> Net-(U1-GPIO46)
- R3 pad 1: +3V3 -> /boot
- R3 pad 2: /reset -> +3V3
- R4 pad 1: /boot -> Net-(U1-GPIO45)
- R4 pad 2: +3V3 -> GND
- R5 pad 1: /io5 -> Net-(J2-CC2)
- R5 pad 2: Net-(Q1-B) -> GND
- R6 pad 1: Net-(U1-GPIO45) -> Net-(J2-CC1)
- R7 pad 1: Net-(U1-GPIO46) -> +3V3
- R7 pad 2: GND -> /io4
- R8 pad 1: Net-(J3-CC2) -> /io5
- R8 pad 2: GND -> Net-(Q1-B)
- R9 pad 1: Net-(J3-CC1) -> /mdb_master_transmit
- U1 pad 1: Net-(U1-LNA_IN/RF) -> unconnected-(U1-LNA_IN/RF-Pad1)
- U1 pad 28: /spics1 -> unconnected-(U1-SPI_CS1/GPIO26-Pad28)
- U1 pad 29: /vdd_spi -> unconnected-(U1-VDD_SPI-Pad29)
- U1 pad 30: /spihd -> unconnected-(U1-SPIHD/GPIO27-Pad30)
- U1 pad 31: /spiwp -> unconnected-(U1-SPIWP/GPIO28-Pad31)
- U1 pad 32: /spics0 -> unconnected-(U1-SPICS0/GPIO29-Pad32)
- U1 pad 33: /spiclk -> unconnected-(U1-SPICLK/GPIO30-Pad33)
- U1 pad 34: /spiq -> unconnected-(U1-SPIQ/GPIO31-Pad34)
- U1 pad 35: /spid -> unconnected-(U1-SPID/GPIO32-Pad35)
- U2 pad 1: GND -> unconnected-(U2-NC-Pad1)
- U2 pad 2: +3V3 -> unconnected-(U2-NC-Pad2)
- U2 pad 3: /vin -> unconnected-(U2-NC-Pad3)
- U2 pad 4: (no net) -> +3V3
- Y1 pad 2: Net-(U1-XTAL_N) -> GND
Routing:
- net GND: track 176.6 -> 0.00 mm, vias 6 -> 0
- net +3V3: track 95.8 -> 0.00 mm, vias 4 -> 0
- net /vin: track 84.1 -> 0.00 mm
- net /io4: track 77.9 -> 0.00 mm
- net /boot: track 58.8 -> 0.00 mm
- net /io5: track 47.7 -> 0.00 mm, vias 1 -> 0
- net /io21: track 46.6 -> 0.00 mm, vias 2 -> 0
- net /u0rxd: track 32.7 -> 0.00 mm, vias 1 -> 0
- net /u0txd: track 32.5 -> 0.00 mm, vias 1 -> 0
- net /io8: track 25.0 -> 0.00 mm, vias 1 -> 0
- net /reset: track 24.7 -> 0.00 mm, vias 1 -> 0
- net /io1: track 24.3 -> 0.00 mm
- net /io9: track 23.0 -> 0.00 mm, vias 1 -> 0
- net /io14: track 23.0 -> 0.00 mm
- net /io2: track 22.0 -> 0.00 mm
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Other:
- board size 41 x 46 mm -> 40 x 46 mm
- board text removed: "on"
