File: kicad/vmflow-mdb-iot-esp32-sim7080g/mdb-slave-esp32s3.kicad_sch (KiCad schematic)
At the start: 41 parts, among them J1 MDB_Connector, J2 USB_C_Receptacle_USB2.0_16P, J3 Conn_02x11_Odd_Even, J4 JAE_SIM_Card_SF72S006, SW1 SW_Push, U1 TLP785, U2 SIM7080G, U3 ESP32-S3FH4R2, U4 TLP785, U5 LM2594HVM-3.3, Y1 Crystal_GND24

Commit message: Connecting power wire
Parts:
- added AE2: Antenna, RF_Antenna:Johanson_2450AT43F0100, symbol Device:Antenna
- added C14: 0.1uF, Capacitor_SMD:C_0603_1608Metric, symbol Device:C
- added C15: 1uF, Capacitor_SMD:C_0603_1608Metric, symbol Device:C
- added C16: 10uF, Capacitor_Tantalum_SMD:CP_EIA-3528-21_Kemet-B, symbol Device:C_Polarized
- added C17, C18, C19, C20: 1.8pf, Capacitor_SMD:C_0603_1608Metric, symbol Device:C
- added D2: LED, LED_SMD:LED_0603_1608Metric, symbol Device:LED
- added J5, J6: Conn_Coaxial, Connector_Coaxial:U.FL_Hirose_U.FL-R-SMT-1_Vertical, symbol Connector:Conn_Coaxial
- added L3, L4: 2.4nh, Inductor_SMD:L_0603_1608Metric, symbol Device:L
- added R1: 1k, Resistor_SMD:R_0603_1608Metric, symbol Device:R
- added TP1: TestPoint, TestPoint:TestPoint_Pad_D1.0mm, symbol Connector:TestPoint
Connections:
- net VBAT is gone; now on net +3V3: U2.34 (VBAT), U2.35 (VBAT)
- net +3V3: now also C14.1, C15.1, C16.1
- net GND: now also C14.2, C15.2, C16.2, C17.1, C18.1, C19.1, C20.1, D2.1 (K), J5.2 (Ext), J6.2 (Ext)
- net io14: now also U2.39 (PWRKEY)
- net io17: now also U2.2 (UART1_RXD)
- net io18: now also U2.1 (UART1_TXD)
- net rf_ant: now reaches U2.32 (RF_ANT)
- net rf_ant: now also C17.2, L3.2
- net netlight: now reaches U2.41 (NETLIGHT)
- net netlight: now also R1.1
- net at U2.42 (STATUS): now also TP1.1
- net gnss_ant: now reaches U2.68 (GNSS_ANT)
- net gnss_ant: now also C20.2, L4.2
- new net: C19.2, J5.1 (In), L4.1
- new net: D2.2 (A), R1.2
- new net: AE2.1 (A), C18.2, J6.1 (In), L3.1
Other:
- moved on the sheet: C13, J4
