File: kicad/mdb-slave-esp32s3-sim7080g/mdb-slave-esp32s3-sim7080g.kicad_sch (KiCad schematic)
At the start: 66 parts, among them J1 MDB_Connector, J2 USB_C_Receptacle_USB2.0_16P, J3 Conn_02x11_Odd_Even, J4 JAE_SIM_Card_SF72S006, J5 Conn_Coaxial, J7 Conn_Coaxial, Q1 NPN, Q2 NPN, Q4 NPN, SW1 SW_Push, U1 TLP785, U2 SIM7080G, U3 ESP32-S3FH4R2, U4 TLP785, U5 LM2594HVM-3.3, Y1 Crystal_GND24

Commit message: Set labels
Parts:
- added D2: LED, LED_SMD:LED_0603_1608Metric, symbol Device:LED
- added R13: 1k, Resistor_SMD:R_0603_1608Metric, symbol Device:R
Connections:
- net +3V3: now also R13.2
- net GND: now also D2.1 (K)
- new net: D2.2 (A), R13.1

Commit message: Reload references
Parts:
- Q1: renamed from Q2; footprint (none) -> Package_TO_SOT_SMD:SOT-23
- Q2: renamed from Q4; footprint (none) -> Package_TO_SOT_SMD:SOT-23
- Q3: renamed from Q1; footprint (none) -> Package_TO_SOT_SMD:SOT-23
- renumbered AE3 to AE1, C22 to C1, C7 to C10, C14 to C11, C16 to C12, C15 to C13, C12 to C14, C3 to C15, C13 to C16, C2 to C17, C19 to C18, C18 to C19, C21 to C2, C17 to C21, C1 to C3, C5 to C4, C6 to C5, C11 to C6, C8 to C7, C9 to C8, C10 to C9, D5 to D1, D4 to D2, D2 to D3, D1 to D4, J2 to J1, J4 to J2, J5 to J4, J7 to J5, J1 to J6, L5 to L1, L4 to L3, L3 to L4, R3 to R1, R7 to R10, R8 to R11, R17 to R12, R18 to R13, R19 to R14, R13 to R15, R2 to R16, R10 to R17, R5 to R18, R12 to R2, R20 to R3, R11 to R4, R21 to R5, R1 to R6, R9 to R7, R4 to R8, R6 to R9, TP4 to TP1, TP1 to TP2, TP2 to TP3, U3 to U1, U5 to U3, U1 to U5

Commit message: UPdating references
Parts:
- L4: LCSC# (none) -> C2042508
Changed lines of the file:
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@@
 	)
 	(symbol
-		(lib_id "Device:L")
-		(at 472.44 288.29 90)
-		(unit 1)
-		(exclude_from_sim no)
-		(in_bom yes)
-		(on_board yes)
-		(dnp no)
-		(fields_autoplaced yes)
-		(property "Reference" "L3"
-			(at 472.44 283.21 90)
-			(effects
-				(font
-					(size 1.27 1.27)
-				)
-			)
-		)
-		(property "Value" "47nh"
-			(at 472.44 285.75 90)
-			(effects
-				(font
-					(size 1.27 1.27)
-				)
-			)
-		)
-		(property "Footprint" "Inductor_SMD:L_0603_1608Metric"
-			(at 472.44 288.29 0)
-			(effects
-				(font
-					(size 1.27 1.27)
-				)
-				(hide yes)
-			)
-		)
-		(property "Datasheet" "~"
-			(at 472.44 288.29 0)
-			(effects
-				(font
-					(size 1.27 1.27)
-				)
-				(hide yes)
-			)
-		)
-		(property "Description" ""
-			(at 472.44 288.29 0)
-			(effects
-				(font
-					(size 1.27 1.27)
-				)
-				(hide yes)
-			)
-		)
-		(property "LCSC#" "C2042508"
-			(at 472.44 288.29 0)
-			(effects
-				(font
-					(size 1.27 1.27)
-				)
-				(hide yes)
-			)
-		)
-		(pin "1"
-		)
-		(pin "2"
-		)
-		(instances
-			(project "mdb-slave-esp32s3"
-				(path "/95980b25-0707-441d-ba83-7f6c6e1d1aaa"
-					(reference "L3")
-					(unit 1)
-				)
-			)
-		)
-	)
-	(symbol
 		(lib_id "Device:C")
 		(at 252.73 264.16 180)
@@
 	)
 	(symbol
+		(lib_id "Device:L")
+		(at 472.44 288.29 90)
+		(unit 1)
+		(exclude_from_sim no)
+		(in_bom yes)
+		(on_board yes)
+		(dnp no)
+		(fields_autoplaced yes)
+		(property "Reference" "L3"
+			(at 472.44 283.21 90)
+			(effects
+				(font
+					(size 1.27 1.27)
+				)
+			)
+		)
+		(property "Value" "47nh"
+			(at 472.44 285.75 90)
+			(effects
+				(font
+					(size 1.27 1.27)
+				)
+			)
+		)
+		(property "Footprint" "Inductor_SMD:L_0603_1608Metric"
+			(at 472.44 288.29 0)
+			(effects
+				(font
+					(size 1.27 1.27)
+				)
+				(hide yes)
+			)
+		)
+		(property "Datasheet" "~"
+			(at 472.44 288.29 0)
+			(effects
+				(font
+					(size 1.27 1.27)
+				)
+				(hide yes)
+			)
+		)
+		(property "Description" ""
+			(at 472.44 288.29 0)
+			(effects
+				(font
+					(size 1.27 1.27)
+				)
+				(hide yes)
+			)
+		)
+		(property "LCSC#" "C2042508"
+			(at 472.44 288.29 0)
+			(effects
+				(font
+					(size 1.27 1.27)
+				)
+				(hide yes)
+			)
+		)
+		(pin "1"
+		)
+		(pin "2"
+		)
+		(instances
+			(project "mdb-slave-esp32s3-sim7080g"
+				(path "/95980b25-0707-441d-ba83-7f6c6e1d1aaa"
+					(reference "L3")
+					(unit 1)
+				)
+			)
+		)
+	)
+	(symbol
 		(lib_id "Device:C")
 		(at 26.67 121.92 180)
@@
 	)
 	(symbol
+		(lib_id "Device:L")
+		(at 474.98 332.74 90)
+		(unit 1)
+		(exclude_from_sim no)
+		(in_bom yes)
+		(on_board yes)
+		(dnp no)
+		(fields_autoplaced yes)
+		(property "Reference" "L4"
+			(at 474.98 327.66 90)
+			(effects
+				(font
+					(size 1.27 1.27)
+				)
+			)
+		)
+		(property "Value" "47nh"
+			(at 474.98 330.2 90)
+			(effects
+				(font
+					(size 1.27 1.27)
+				)
+			)
+		)
+		(property "Footprint" "Inductor_SMD:L_0603_1608Metric"
+			(at 474.98 332.74 0)
+			(effects
+				(font
+					(size 1.27 1.27)
+				)
+				(hide yes)
+			)
+		)
+		(property "Datasheet" "~"
+			(at 474.98 332.74 0)
+			(effects
+				(font
+					(size 1.27 1.27)
+				)
+				(hide yes)
+			)
+		)
+		(property "Description" ""
+			(at 474.98 332.74 0)
+			(effects
+				(font
+					(size 1.27 1.27)
+				)
+				(hide yes)
+			)
+		)
+		(property "LCSC#" "C2042508"
+			(at 474.98 332.74 0)
+			(effects
+				(font
+					(size 1.27 1.27)
+				)
+				(hide yes)
+			)
+		)
+		(pin "1"
+		)
+		(pin "2"
+		)
+		(instances
+			(project "mdb-slave-esp32s3-sim7080g"
+				(path "/95980b25-0707-441d-ba83-7f6c6e1d1aaa"
+					(reference "L4")
+					(unit 1)
+				)
+			)
+		)
+	)
+	(symbol
 		(lib_id "Device:R")
 		(at 182.88 130.81 90)
@@
 					(unit 1)
 				)
-			)
-		)
-	)
-	(symbol
-		(lib_id "Device:L")
-		(at 474.98 332.74 90)
-		(unit 1)
-		(exclude_from_sim no)
-		(in_bom yes)
-		(on_board yes)
-		(dnp no)
-		(fields_autoplaced yes)
-		(property "Reference" "L4"
-			(at 474.98 327.66 90)
-			(effects
-				(font
-					(size 1.27 1.27)
-				)
-			)
-		)
-		(property "Value" "47nh"
-			(at 474.98 330.2 90)
-			(effects
-				(font
-					(size 1.27 1.27)
-				)
-			)
-		)
-		(property "Footprint" "Inductor_SMD:L_0603_1608Metric"
-			(at 474.98 332.74 0)
-			(effects
-				(font
-					(size 1.27 1.27)
-				)
-				(hide yes)
-			)
-		)
-		(property "Datasheet" "~"
-			(at 474.98 332.74 0)
-			(effects
-				(font
-					(size 1.27 1.27)
-				)
-				(hide yes)
-			)
-		)
-		(property "Description" ""
-			(at 474.98 332.74 0)
-			(effects
-				(font
-					(size 1.27 1.27)
-				)
-				(hide yes)
-			)
-		)
-		(property "LCSC#" ""
-			(at 474.98 332.74 0)
-			(effects
-				(font
-					(size 1.27 1.27)
-				)
-				(hide yes)
-			)
-		)
-		(pin "1"
-		)
-		(pin "2"
-		)
-		(instances
-			(project "mdb-slave-esp32s3"
-				(path "/95980b25-0707-441d-ba83-7f6c6e1d1aaa"
-					(reference "L4")
-					(unit 1)
-				)

Commit message: Refacting
Parts:
- added TP4: TestPoint, TestPoint:TestPoint_Pad_D1.0mm, symbol Connector:TestPoint
Connections:
- net vin: now also TP4.1
Other:
- moved on the sheet: TP1, TP2, TP3
Changed lines of the file:
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@@
 	)
 	(junction
+		(at 407.67 147.32)
+		(diameter 0)
+		(color 0 0 0 0)
+	)
+	(junction
 		(at 81.28 144.78)
 		(diameter 0)
@@
 	(wire
 		(pts
-			(xy 227.33 275.59) (xy 236.22 275.59)
+			(xy 227.33 275.59) (xy 242.57 275.59)
 		)
 		(stroke
@@
 	(wire
 		(pts
+			(xy 414.02 147.32) (xy 407.67 147.32)
+		)
+		(stroke
+			(width 0)
+			(type default)
+		)
+	)
+	(wire
+		(pts
 			(xy 209.55 30.48) (xy 201.93 30.48)
 		)
@@
 	(wire
 		(pts
-			(xy 227.33 283.21) (xy 217.17 283.21)
+			(xy 236.22 283.21) (xy 217.17 283.21)
 		)
 		(stroke
@@
 	(wire
 		(pts
-			(xy 78.74 38.1) (xy 78.74 36.83)
-		)
-		(stroke
-			(width 0)
-			(type default)
-		)
-	)
-	(wire
-		(pts
 			(xy 86.36 120.65) (xy 86.36 123.19)
 		)
@@
 	)
 	(symbol
+		(lib_id "Connector:TestPoint")
+		(at 341.63 144.78 0)
+		(unit 1)
+		(exclude_from_sim no)
+		(in_bom yes)
+		(on_board yes)
+		(dnp no)
+		(fields_autoplaced yes)
+		(property "Reference" "TP4"
+			(at 344.17 140.2079 0)
+			(effects
+				(font
+					(size 1.27 1.27)
+				)
+				(justify left)
+			)
+		)
+		(property "Value" "TestPoint"
+			(at 344.17 142.7479 0)
+			(effects
+				(font
+					(size 1.27 1.27)
+				)
+				(justify left)
+			)
+		)
+		(property "Footprint" "TestPoint:TestPoint_Pad_D1.0mm"
+			(at 346.71 144.78 0)
+			(effects
+				(font
+					(size 1.27 1.27)
+				)
+				(hide yes)
+			)
+		)
+		(property "Datasheet" "~"
+			(at 346.71 144.78 0)
+			(effects
+				(font
+					(size 1.27 1.27)
+				)
+				(hide yes)
+			)
+		)
+		(property "Description" "test point"
+			(at 341.63 144.78 0)
+			(effects
+				(font
+					(size 1.27 1.27)
+				)
+				(hide yes)
+			)
+		)
+		(pin "1"
+		)
+		(instances
+			(project "mdb-slave-esp32s3-sim7080g"
+				(path "/95980b25-0707-441d-ba83-7f6c6e1d1aaa"
+					(reference "TP4")
+					(unit 1)
+				)
+			)
+		)
+	)
+	(symbol
 		(lib_id "Graphic:Logo_Open_Hardware_Small")
 		(at 35.56 35.56 0)
@@
 	(symbol
 		(lib_id "Connector:TestPoint")
-		(at 236.22 275.59 270)
+		(at 242.57 275.59 0)
 		(unit 1)
 		(exclude_from_sim no)
@@
 		(fields_autoplaced yes)
 		(property "Reference" "TP3"
-			(at 241.3 274.3199 90)
+			(at 245.11 271.0179 0)
 			(effects
 				(font
@@
 		)
 		(property "Value" "TestPoint"
-			(at 241.3 276.8599 90)
+			(at 245.11 273.5579 0)
 			(effects
 				(font
@@
 		)
 		(property "Footprint" "TestPoint:TestPoint_Pad_D1.0mm"
-			(at 236.22 280.67 0)
+			(at 247.65 275.59 0)
 			(effects
 				(font
@@
 		)
 		(property "Datasheet" "~"
-			(at 236.22 280.67 0)
+			(at 247.65 275.59 0)
 			(effects
 				(font
@@
 		)
 		(property "Description" "test point"
-			(at 236.22 275.59 0)
+			(at 242.57 275.59 0)
 			(effects
 				(font
@@
 	(symbol
 		(lib_id "Connector:TestPoint")
-		(at 78.74 36.83 0)
+		(at 407.67 147.32 0)
 		(unit 1)
 		(exclude_from_sim no)
@@
 		(fields_autoplaced yes)
 		(property "Reference" "TP1"
-			(at 81.28 32.2579 0)
+			(at 410.21 142.7479 0)
 			(effects
 				(font
@@
 		)
 		(property "Value" "TestPoint"
-			(at 81.28 34.7979 0)
+			(at 410.21 145.2879 0)
 			(effects
 				(font
@@
 		)
 		(property "Footprint" "TestPoint:TestPoint_Pad_D1.0mm"
-			(at 83.82 36.83 0)
+			(at 412.75 147.32 0)
 			(effects
 				(font
@@
 		)
 		(property "Datasheet" "~"
-			(at 83.82 36.83 0)
+			(at 412.75 147.32 0)
 			(effects
 				(font
@@
 		)
 		(property "Description" "test point"
-			(at 78.74 36.83 0)
+			(at 407.67 147.32 0)
 			(effects
 				(font
@@
 		)
 		(instances
-			(project "mdb-slave-esp32s3"
+			(project "mdb-slave-esp32s3-sim7080g"
 				(path "/95980b25-0707-441d-ba83-7f6c6e1d1aaa"
 					(reference "TP1")
@@
 	(symbol
 		(lib_id "power:+3V3")
-		(at 407.67 147.32 270)
+		(at 414.02 147.32 270)
 		(unit 1)
 		(exclude_from_sim no)
@@
 		(fields_autoplaced yes)
 		(property "Reference" "#PWR049"
-			(at 403.86 147.32 0)
+			(at 410.21 147.32 0)
 			(effects
 				(font
@@
 		)
 		(property "Value" "+3V3"
-			(at 411.48 147.3199 90)
+			(at 417.83 147.3199 90)
 			(effects
 				(font
@@
 		)
 		(property "Footprint" ""
-			(at 407.67 147.32 0)
+			(at 414.02 147.32 0)
 			(effects
 				(font
@@
 		)
 		(property "Datasheet" ""
-			(at 407.67 147.32 0)
+			(at 414.02 147.32 0)
 			(effects
 				(font
@@
 		)
 		(property "Description" ""
-			(at 407.67 147.32 0)
+			(at 414.02 147.32 0)
 			(effects
 				(font
@@
 	)
 	(symbol
-		(lib_id "power:+3V3")
-		(at 78.74 38.1 180)
-		(unit 1)
-		(exclude_from_sim no)
-		(in_bom yes)
-		(on_board yes)
-		(dnp no)
-		(fields_autoplaced yes)
-		(property "Reference" "#PWR08"
-			(at 78.74 34.29 0)
-			(effects
-				(font
-					(size 1.27 1.27)
-				)
-				(hide yes)
-			)
-		)
-		(property "Value" "+3V3"
-			(at 78.74 43.18 0)
-			(effects
-				(font
-					(size 1.27 1.27)
-				)
-			)
-		)
-		(property "Footprint" ""
-			(at 78.74 38.1 0)
-			(effects
-				(font
-					(size 1.27 1.27)
-				)
-				(hide yes)
-			)
-		)
-		(property "Datasheet" ""
-			(at 78.74 38.1 0)
-			(effects
-				(font
-					(size 1.27 1.27)
-				)
-				(hide yes)
-			)
-		)
-		(property "Description" ""
-			(at 78.74 38.1 0)
-			(effects
-				(font
-					(size 1.27 1.27)
-				)
-				(hide yes)
-			)
-		)
-		(pin "1"
-		)
-		(instances
-			(project "mdb-slave-esp32s3"
-				(path "/95980b25-0707-441d-ba83-7f6c6e1d1aaa"
-					(reference "#PWR08")
-					(unit 1)
-				)
-			)
-		)
-	)
-	(symbol
 		(lib_id "power:GND")
 		(at 259.08 283.21 0)
@@
 	(symbol
 		(lib_id "Connector:TestPoint")
-		(at 227.33 283.21 270)
+		(at 236.22 283.21 0)
 		(unit 1)
 		(exclude_from_sim no)
@@
 		(fields_autoplaced yes)
 		(property "Reference" "TP2"
-			(at 232.41 281.9399 90)
+			(at 238.76 278.6379 0)
 			(effects
 				(font
@@
 		)
 		(property "Value" "TestPoint"
-			(at 232.41 284.4799 90)
+			(at 238.76 281.1779 0)
 			(effects
 				(font
@@
 		)
 		(property "Footprint" "TestPoint:TestPoint_Pad_D1.0mm"
-			(at 227.33 288.29 0)
+			(at 241.3 283.21 0)
 			(effects
 				(font
@@
 		)
 		(property "Datasheet" "~"
-			(at 227.33 288.29 0)
+			(at 241.3 283.21 0)
 			(effects
 				(font
@@
 		)
 		(property "Description" "test point"
-			(at 227.33 283.21 0)
+			(at 236.22 283.21 0)
 			(effects
 				(font

Commit message: Initial organization
Parts:
- removed D3: LED, LED_SMD:LED_0603_1608Metric, symbol Device:LED
- removed R15: 1k, Resistor_SMD:R_0603_1608Metric, symbol Device:R

Commit message: PCB routing
Parts:
- added H1, H2: MountingHole, MountingHole:MountingHole_2.1mm, symbol Mechanical:MountingHole
Changed lines of the file:
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@@
 	)
 	(symbol
+		(lib_id "Mechanical:MountingHole")
+		(at 518.16 295.91 0)
+		(unit 1)
+		(exclude_from_sim no)
+		(in_bom no)
+		(on_board yes)
+		(dnp no)
+		(fields_autoplaced yes)
+		(property "Reference" "H2"
+			(at 520.7 294.6399 0)
+			(effects
+				(font
+					(size 1.27 1.27)
+				)
+				(justify left)
+			)
+		)
+		(property "Value" "MountingHole"
+			(at 520.7 297.1799 0)
+			(effects
+				(font
+					(size 1.27 1.27)
+				)
+				(justify left)
+			)
+		)
+		(property "Footprint" "MountingHole:MountingHole_2.1mm"
+			(at 518.16 295.91 0)
+			(effects
+				(font
+					(size 1.27 1.27)
+				)
+				(hide yes)
+			)
+		)
+		(property "Datasheet" "~"
+			(at 518.16 295.91 0)
+			(effects
+				(font
+					(size 1.27 1.27)
+				)
+				(hide yes)
+			)
+		)
+		(property "Description" "Mounting Hole without connection"
+			(at 518.16 295.91 0)
+			(effects
+				(font
+					(size 1.27 1.27)
+				)
+				(hide yes)
+			)
+		)
+		(instances
+			(project "mdb-slave-esp32s3-sim7080g"
+				(path "/95980b25-0707-441d-ba83-7f6c6e1d1aaa"
+					(reference "H2")
+					(unit 1)
+				)
+			)
+		)
+	)
+	(symbol
 		(lib_id "Simulation_SPICE:NPN")
 		(at 124.46 260.35 0)
@@
 					(unit 1)
 				)
+			)
+		)
+	)
+	(symbol
+		(lib_id "Mechanical:MountingHole")
+		(at 518.16 289.56 0)
+		(unit 1)
+		(exclude_from_sim no)
+		(in_bom no)
+		(on_board yes)
+		(dnp no)
+		(fields_autoplaced yes)
+		(property "Reference" "H1"
+			(at 520.7 288.2899 0)
+			(effects
+				(font
+					(size 1.27 1.27)
+				)
+				(justify left)
+			)
+		)
+		(property "Value" "MountingHole"
+			(at 520.7 290.8299 0)
+			(effects
+				(font
+					(size 1.27 1.27)
+				)
+				(justify left)
+			)
+		)
+		(property "Footprint" "MountingHole:MountingHole_2.1mm"
+			(at 518.16 289.56 0)
+			(effects
+				(font
+					(size 1.27 1.27)
+				)
+				(hide yes)
+			)
+		)
+		(property "Datasheet" "~"
+			(at 518.16 289.56 0)
+			(effects
+				(font
+					(size 1.27 1.27)
+				)
+				(hide yes)
+			)
+		)
+		(property "Description" "Mounting Hole without connection"
+			(at 518.16 289.56 0)
+			(effects
+				(font
+					(size 1.27 1.27)
+				)
+				(hide yes)
+			)
+		)
+		(instances
+			(project ""
+				(path "/95980b25-0707-441d-ba83-7f6c6e1d1aaa"
+					(reference "H1")
+					(unit 1)
+				)

Commit message: Refacting production components
Connections:
- net GND: now also J3.2 (Pin_2)
- net reset: no longer names the net of C3.1, R1.2, U1.4 (CHIP_PU/RESET)
- net reset: no longer J3.2 (Pin_2)
Changed lines of the file:
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@@
 	)
 	(junction
-		(at 86.36 123.19)
-		(diameter 0)
-		(color 0 0 0 0)
-	)
-	(junction
 		(at 269.24 152.4)
 		(diameter 0)
@@
 	(wire
 		(pts
-			(xy 86.36 123.19) (xy 99.06 123.19)
+			(xy 63.5 123.19) (xy 99.06 123.19)
 		)
 		(stroke
@@
 	(wire
 		(pts
-			(xy 63.5 123.19) (xy 86.36 123.19)
-		)
-		(stroke
-			(width 0)
-			(type default)
-		)
-	)
-	(wire
-		(pts
 			(xy 318.77 66.04) (xy 318.77 68.58)
 		)
@@
 	(wire
 		(pts
-			(xy 403.86 69.85) (xy 400.05 69.85)
+			(xy 411.48 69.85) (xy 400.05 69.85)
 		)
 		(stroke
@@
 	(wire
 		(pts
-			(xy 86.36 120.65) (xy 86.36 123.19)
-		)
-		(stroke
-			(width 0)
-			(type default)
-		)
-	)
-	(wire
-		(pts
 			(xy 157.48 306.07) (xy 166.37 306.07)
 		)
@@
 		)
 	)
-	(label "reset"
-		(at 86.36 120.65 0)
-		(effects
-			(font
-				(size 1.27 1.27)
-			)
-			(justify left bottom)
-		)
-	)
 	(label "io18"
 		(at 381 92.71 0)
@@
 		)
 	)
-	(label "reset"
-		(at 403.86 69.85 0)
-		(effects
-			(font
-				(size 1.27 1.27)
-			)
-			(justify left bottom)
-		)
-	)
 	(label "boot"
 		(at 167.64 129.54 0)
@@
 					(unit 1)
 				)
+			)
+		)
+	)
+	(symbol
+		(lib_id "power:GND")
+		(at 411.48 69.85 90)
+		(unit 1)
+		(exclude_from_sim no)
+		(in_bom yes)
+		(on_board yes)
+		(dnp no)
+		(fields_autoplaced yes)
+		(property "Reference" "#PWR08"
+			(at 417.83 69.85 0)
+			(effects
+				(font
+					(size 1.27 1.27)
+				)
+				(hide yes)
+			)
+		)
+		(property "Value" "GND"
+			(at 415.29 69.85 90)
+			(effects
+				(font
+					(size 1.27 1.27)
+				)
+				(justify right)
+			)
+		)
+		(property "Footprint" ""
+			(at 411.48 69.85 0)
+			(effects
+				(font
+					(size 1.27 1.27)
+				)
+				(hide yes)
+			)
+		)
+		(property "Datasheet" ""
+			(at 411.48 69.85 0)
+			(effects
+				(font
+					(size 1.27 1.27)
+				)
+				(hide yes)
+			)
+		)
+		(property "Description" ""
+			(at 411.48 69.85 0)
+			(effects
+				(font
+					(size 1.27 1.27)
+				)
+				(hide yes)
+			)
+		)
+		(pin "1"
+		)
+		(instances
+			(project "mdb-slave-esp32s3-sim7080g"
+				(path "/95980b25-0707-441d-ba83-7f6c6e1d1aaa"
+					(reference "#PWR08")
+					(unit 1)
+				)

Commit message: updating production components
Parts:
- removed C18: 27pf, Capacitor_SMD:C_0603_1608Metric, symbol Device:C
- C19: value 27pf -> 1.8pf; LCSC# (none) -> C376773
- C2: value NC -> 1.8pf
- C20, C21, TP1, TP2, TP3, TP4: now left out of the parts list
- L3: value 47nh -> 5.6nh; LCSC# C2042508 -> C6652920
- L4: value 47nh -> 3.9nh; LCSC# C2042508 -> C317982
- R2, R3: value 10K -> 10k
Connections:
- net GND: now also L1.1; no longer C1.1
- net at J4.1 (In), L3.1: now also C2.2
- new net: AE1.1 (A), C1.1, L1.2
- new net: C1.2, U1.1 (LNA_IN/RF)
Other:
- moved on the sheet: C1, C19, C20, C21, L1
