File: kicad/mdb-slave-esp32s3-sim7080g/mdb-slave-esp32s3-sim7080g.kicad_sch (KiCad schematic)
At the start: 82 parts, among them J1 USB_C_Receptacle_USB2.0_16P, J2 JAE_SIM_Card_SF72S006, J3 Conn_01x03_Pin, J4 Conn_Coaxial, J5 Conn_Coaxial, J6 MDB_Connector, J7 Conn_01x03_Pin, J8 Conn_01x04_Pin, Q1 MMBT3904, Q2 MMBT3904, Q3 MMBT3904, Q4 MMBT3904, Q5 MMBT3904, Q6 MMBT3904, Q7 MMBT3904, SW1 SW_Push, U1 ESP32-S3FH4R2, U2 SIM7080G, U3 LM2594HVM-3.3, U4 TLP785, U5 TLP785, Y1 Crystal_GND24

Commit message: tlp185 to tlp785
Parts:
- U4, U5: LCSC# C128776 -> C45445
Changed lines of the file:
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@@
 			)
 		)
-		(property "LCSC#" "C128776"
+		(property "LCSC#" "C45445"
 			(at 518.16 107.95 0)
 			(effects
@@
 			)
 		)
-		(property "LCSC#" "C128776"
+		(property "LCSC#" "C45445"
 			(at 518.16 123.19 0)
 			(effects
