File: kicad/mdb-slave-esp32s3-sim7080g/mdb-slave-esp32s3-sim7080g.kicad_sch (KiCad schematic)
At the start: 82 parts, among them J1 USB_C_Receptacle_USB2.0_16P, J2 JAE_SIM_Card_SF72S006, J3 Conn_01x03_Pin, J4 Conn_Coaxial, J5 Conn_Coaxial, J6 MDB_Connector, J7 Conn_01x03_Pin, J8 Conn_01x04_Pin, Q1 MMBT3904, Q2 MMBT3904, Q3 MMBT3904, Q4 MMBT3904, Q5 MMBT3904, Q6 MMBT3904, Q7 MMBT3904, SW1 SW_Push, U1 ESP32-S3FH4R2, U2 SIM7080G, U3 LM2594HVM-3.3, U4 TLP785, U5 TLP785, Y1 Crystal_GND24

Commit message: fix(hardware): standardize Value field notation in schematics
4K7→4.7k, 22ohm→22R, 470ohm→470R, 1.8pf→1.8pF, 2.4nh→2.4nH,
5.6nh→5.6nH, 3.9nh→3.9nH, Crystal_GND24→40MHz, FerriteBead_Small→FerriteBead

Co-Authored-By: Claude Sonnet 4.6 <noreply@anthropic.com>
Parts:
- C1, C19, C2: value 1.8pf -> 1.8pF
- FB1: value FerriteBead_Small -> FerriteBead
- L1: value 2.4nh -> 2.4nH
- L3: value 5.6nh -> 5.6nH
- L4: value 3.9nh -> 3.9nH
- R12, R13, R14: value 22ohm -> 22R
- R15, R19, R21, R23, R24, R25, R4, R5, R6: value 4K7 -> 4.7k
- R16, R18: value 470ohm -> 470R
- Y1: value Crystal_GND24 -> 40MHz
Changed lines of the file:
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@@
 			)
 		)
-		(property "Value" "4K7"
+		(property "Value" "4.7k"
 			(at 91.44 365.7599 0)
 			(effects
@@
 			)
 		)
-		(property "Value" "4K7"
+		(property "Value" "4.7k"
 			(at 350.52 54.61 90)
 			(effects
@@
 			)
 		)
-		(property "Value" "4K7"
+		(property "Value" "4.7k"
 			(at 421.64 71.1199 0)
 			(effects
@@
 			)
 		)
-		(property "Value" "4K7"
+		(property "Value" "4.7k"
 			(at 434.34 68.5799 0)
 			(effects
@@
 			)
 		)
-		(property "Value" "470ohm"
+		(property "Value" "470R"
 			(at 533.4 130.8099 0)
 			(effects
@@
 			)
 		)
-		(property "Value" "1.8pf"
+		(property "Value" "1.8pF"
 			(at 424.18 295.9099 0)
 			(effects
@@
 			)
 		)
-		(property "Value" "4K7"
+		(property "Value" "4.7k"
 			(at 513.08 289.56 90)
 			(effects
@@
 			)
 		)
-		(property "Value" "5.6nh"
+		(property "Value" "5.6nH"
 			(at 427.99 285.75 90)
 			(effects
@@
 			)
 		)
-		(property "Value" "1.8pf"
+		(property "Value" "1.8pF"
 			(at 33.0201 119.38 0)
 			(effects
@@
 			)
 		)
-		(property "Value" "3.9nh"
+		(property "Value" "3.9nH"
 			(at 430.53 330.2 90)
 			(effects
@@
 			)
 		)
-		(property "Value" "1.8pf"
+		(property "Value" "1.8pF"
 			(at 424.18 340.3599 0)
 			(effects
@@
 			)
 		)
-		(property "Value" "4K7"
+		(property "Value" "4.7k"
 			(at 533.4 233.6799 0)
 			(effects
@@
 			)
 		)
-		(property "Value" "4K7"
+		(property "Value" "4.7k"
 			(at 90.17 250.19 90)
 			(effects
@@
 			)
 		)
-		(property "Value" "4K7"
+		(property "Value" "4.7k"
 			(at 83.82 326.3899 0)
 			(effects
@@
 			)
 		)
-		(property "Value" "FerriteBead_Small"
+		(property "Value" "FerriteBead"
 			(at 162.5219 44.45 90)
 			(effects
@@
 			)
 		)
-		(property "Value" "22ohm"
+		(property "Value" "22R"
 			(at 300.99 302.26 90)
 			(effects
@@
 			)
 		)
-		(property "Value" "Crystal_GND24"
+		(property "Value" "40MHz"
 			(at 93.98 136.0168 90)
 			(effects
@@
 			)
 		)
-		(property "Value" "22ohm"
+		(property "Value" "22R"
 			(at 323.85 299.72 90)
 			(effects
@@
 			)
 		)
-		(property "Value" "470ohm"
+		(property "Value" "470R"
 			(at 505.46 101.6 90)
 			(effects
@@
 			)
 		)
-		(property "Value" "4K7"
+		(property "Value" "4.7k"
 			(at 525.78 191.7699 0)
 			(effects
@@
 			)
 		)
-		(property "Value" "22ohm"
+		(property "Value" "22R"
 			(at 316.23 309.88 90)
 			(effects
@@
 			)
 		)
-		(property "Value" "2.4nh"
+		(property "Value" "2.4nH"
 			(at 24.13 121.92 90)
 			(effects

Commit message: fix(kicad): resolve ERC violations in mdb-slave-esp32s3 schematics
All ERC validations pass now on both sim7080g and base variants.

Co-Authored-By: Claude Sonnet 5 <noreply@anthropic.com>
Connections:
- net io1: no longer names the net of U1.6 (GPIO1/ADC1_CH0)
- net io2: no longer names the net of U1.7 (GPIO2/ADC1_CH1)
- net io7: no longer names the net of U1.12 (GPIO7/ADC1_CH6)
- net netlight: no longer names the net of U2.41 (NETLIGHT)
- net u0rxd: no longer names the net of U1.50 (U0RXD/PROG/GPIO44)
- net u0txd: no longer names the net of U1.49 (U0TXD/PROG/GPIO43)
- no-connect marks 31 -> 70
