File: kicad/mdb-slave-esp32s3-sim7080g/mdb-slave-esp32s3-sim7080g.kicad_pcb (KiCad board)
At the start: 2 copper layers, 65 x 40 mm, 82 parts, among them J1 USB_C_Receptacle_USB2.0_16P, J2 JAE_SIM_Card_SF72S006, J3 Conn_01x03_Pin, J4 Conn_Coaxial, J5 Conn_Coaxial, J6 MDB_Connector, J7 Conn_01x03_Pin, J8 Conn_01x04_Pin, Q1 MMBT3904, Q2 MMBT3904, Q3 MMBT3904, Q4 MMBT3904, Q5 MMBT3904, Q6 MMBT3904, Q7 MMBT3904, SW1 SW_Push, U1 ESP32-S3FH4R2, U2 SIM7080G, U3 LM2594HVM-3.3, U4 TLP785, U5 TLP785, Y1 Crystal_GND24

Commit message: routing...
Routing:
- net GND: track 218.6 -> 206.1 mm, vias 26 -> 27
Changed lines of the file:
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@@
 	)
 	(segment
-		(start 189.6426 84.1326)
-		(end 191.7 86.19)
-		(width 0.508)
-		(layer "F.Cu")
-		(net 3)
-	)
-	(segment
 		(start 214.37 97.9925)
 		(end 215.52 97.9925)
@@
 	)
 	(segment
-		(start 183.38 90.068334)
-		(end 184.86 88.588334)
-		(width 0.508)
-		(layer "F.Cu")
-		(net 3)
-	)
-	(segment
 		(start 229.3 98.5725)
 		(end 229.3 100.13)
@@
 	)
 	(segment
+		(start 183.38 90.068334)
+		(end 184.32 90.068334)
+		(width 0.508)
+		(layer "F.Cu")
+		(net 3)
+	)
+	(segment
 		(start 195.2 107.559285)
 		(end 196.025 106.734285)
@@
 	)
 	(segment
-		(start 184.86 88.588334)
-		(end 184.86 85.39337)
-		(width 0.508)
-		(layer "F.Cu")
-		(net 3)
-	)
-	(segment
 		(start 216.0274 107.6851)
 		(end 221.113015 107.6851)
@@
 	)
 	(segment
-		(start 186.12077 84.1326)
-		(end 189.6426 84.1326)
-		(width 0.508)
-		(layer "F.Cu")
-		(net 3)
-	)
-	(segment
 		(start 222.6224 121.0626)
 		(end 225.1076 121.0626)
@@
 	)
 	(segment
-		(start 184.86 85.39337)
-		(end 186.12077 84.1326)
-		(width 0.508)
-		(layer "F.Cu")
-		(net 3)
-	)
-	(segment
 		(start 188.75 97.17)
 		(end 189.375 97.17)
@@
 	)
 	(via
+		(at 184.32 90.068334)
+		(size 0.8)
+		(drill 0.4)
+		(layers "F.Cu" "B.Cu")
+		(net 3)
+	)
+	(via
 		(at 224.85 108.38)
 		(size 0.8)
@@
 	)
 	(zone
-		(net 3)
-		(net_name "GND")
-		(layer "F.Cu")
-		(name "$teardrop_padvia$")
-		(hatch none 0.1)
-		(priority 30001)
-		(attr
-			(teardrop
-				(type padvia)
-			)
-		)
-		(connect_pads yes
-			(clearance 0)
-		)
-		(min_thickness 0.0254)
-		(filled_areas_thickness no)
-		(fill yes
-			(thermal_gap 0.5)
-			(thermal_bridge_width 0.5)
-			(island_removal_mode 1)
-			(island_area_min 10)
-		)
-		(polygon
-			(pts
-				(xy 190.082878 84.213668) (xy 189.723668 84.572878) (xy 190.35 86.254213) (xy 191.700707 86.190707)
-				(xy 191.485911 84.561698)
-			)
-		)
-	)
-	(zone
 		(net 22)
 		(net_name "/io10")
@@
 		(name "$teardrop_padvia$")
 		(hatch none 0.1)
-		(priority 30010)
+		(priority 30009)
 		(attr
 			(teardrop
@@
 	)
 	(zone
-		(net 12)
-		(net_name "/mdb_master_receive")
+		(net 96)
+		(net_name "/dex_rx")
 		(layer "F.Cu")
 		(name "$teardrop_padvia$")
 		(hatch none 0.1)
-		(priority 30004)
+		(priority 30011)
 		(attr
 			(teardrop
@@
 		(polygon
 			(pts
-				(xy 189.367438 89.963983) (xy 189.226017 89.822562) (xy 187.714088 90.061698) (xy 187.499293 91.690707)
-				(xy 188.85 91.754214)
+				(xy 173.96453 94.549232) (xy 174.105951 94.407811) (xy 174.423882 93.669056) (xy 173.924293 93.060007)
+				(xy 173.426118 93.669056)
 			)
 		)
 	)
 	(zone
-		(net 10)
-		(net_name "/mdb_master_transmit")
+		(net 128)
+		(net_name "/dex_tx")
 		(layer "F.Cu")
 		(name "$teardrop_padvia$")
 		(hatch none 0.1)
-		(priority 30002)
+		(priority 30004)
 		(attr
 			(teardrop
@@
 		(polygon
 			(pts
-				(xy 193.424885 93.558569) (xy 193.568569 93.414885) (xy 193.05 91.625786) (xy 191.699293 91.689293)
-				(xy 191.914088 93.318301)
+				(xy 170.899084 93.945209) (xy 171.040505 94.08663) (xy 171.910057 93.924185) (xy 171.925707 93.060007)
+				(xy 171.325 92.812185)
 			)
 		)
 	)
 	(zone
-		(net 96)
-		(net_name "/dex_rx")
+		(net 11)
+		(net_name "/mdb_communications_common")
 		(layer "F.Cu")
 		(name "$teardrop_padvia$")
 		(hatch none 0.1)
-		(priority 30012)
+		(priority 30002)
 		(attr
 			(teardrop
@@
 		(polygon
 			(pts
-				(xy 173.96453 94.549232) (xy 174.105951 94.407811) (xy 174.423882 93.669056) (xy 173.924293 93.060007)
-				(xy 173.426118 93.669056)
+				(xy 197.626017 93.557438) (xy 197.767438 93.416017) (xy 197.25 91.625786) (xy 195.899293 91.689293)
+				(xy 196.114087 93.318301)
 			)
 		)
 	)
 	(zone
-		(net 2)
-		(net_name "+3V3")
+		(net 12)
+		(net_name "/mdb_master_receive")
 		(layer "F.Cu")
 		(name "$teardrop_padvia$")
 		(hatch none 0.1)
-		(priority 30006)
+		(priority 30003)
 		(attr
 			(teardrop
@@
 		(polygon
 			(pts
-				(xy 175.040505 102.466227) (xy 174.899084 102.607648) (xy 175.325 103.740671) (xy 175.925707 103.49285)
-				(xy 175.910057 102.628672)
+				(xy 189.367438 89.963983) (xy 189.226017 89.822562) (xy 187.714088 90.061698) (xy 187.499293 91.690707)
+				(xy 188.85 91.754214)
 			)
 		)
@@
 		(name "$teardrop_padvia$")
 		(hatch none 0.1)
-		(priority 30005)
-		(attr
-			(teardrop
-				(type padvia)
-			)
-		)
-		(connect_pads yes
-			(clearance 0)
-		)
-		(min_thickness 0.0254)
-		(filled_areas_thickness no)
-		(fill yes
-			(thermal_gap 0.5)
-			(thermal_bridge_width 0.5)
-			(island_removal_mode 1)
-			(island_area_min 10)
-		)
-		(polygon
-			(pts
-				(xy 170.899084 93.945209) (xy 171.040505 94.08663) (xy 171.910057 93.924185) (xy 171.925707 93.060007)
-				(xy 171.325 92.812185)
-			)
-		)
-	)
-	(zone
-		(net 7)
-		(net_name "/vin")
-		(layer "F.Cu")
-		(name "$teardrop_padvia$")
-		(hatch none 0.1)
-		(priority 30000)
+		(priority 30006)
 		(attr
 			(teardrop
@@
 		(polygon
 			(pts
-				(xy 189.38033 88.423883) (xy 189.733883 88.07033) (xy 188.849999 86.125786) (xy 187.499293 86.189293)
-				(xy 187.735785 87.839999)
+				(xy 172.809495 94.08663) (xy 172.950916 93.945209) (xy 172.525 92.812186) (xy 171.924293 93.060007)
+				(xy 171.939943 93.924185)
 			)
 		)
@@
 	)
 	(zone
-		(net 128)
-		(net_name "/dex_tx")
+		(net 2)
+		(net_name "+3V3")
 		(layer "F.Cu")
 		(name "$teardrop_padvia$")
 		(hatch none 0.1)
-		(priority 30007)
+		(priority 30008)
 		(attr
 			(teardrop
@@
 		(polygon
 			(pts
-				(xy 172.809495 94.08663) (xy 172.950916 93.945209) (xy 172.525 92.812186) (xy 171.924293 93.060007)
-				(xy 171.939943 93.924185)
+				(xy 176.025 102.028672) (xy 175.825 102.028672) (xy 175.426118 102.883801) (xy 175.925 103.493143)
+				(xy 176.423882 102.883801)
 			)
 		)
 	)
 	(zone
-		(net 11)
-		(net_name "/mdb_communications_common")
+		(net 10)
+		(net_name "/mdb_master_transmit")
 		(layer "F.Cu")
 		(name "$teardrop_padvia$")
 		(hatch none 0.1)
-		(priority 30003)
+		(priority 30001)
 		(attr
 			(teardrop
@@
 		(polygon
 			(pts
-				(xy 197.626017 93.557438) (xy 197.767438 93.416017) (xy 197.25 91.625786) (xy 195.899293 91.689293)
-				(xy 196.114087 93.318301)
+				(xy 193.424885 93.558569) (xy 193.568569 93.414885) (xy 193.05 91.625786) (xy 191.699293 91.689293)
+				(xy 191.914088 93.318301)
 			)
 		)
 	)
 	(zone
-		(net 26)
-		(net_name "/io11")
+		(net 2)
+		(net_name "+3V3")
 		(layer "F.Cu")
 		(name "$teardrop_padvia$")
 		(hatch none 0.1)
-		(priority 30011)
+		(priority 30007)
 		(attr
 			(teardrop
@@
 		(polygon
 			(pts
-				(xy 171.825 104.955614) (xy 172.025 104.955614) (xy 172.423882 104.100485) (xy 171.925 103.491143)
-				(xy 171.426118 104.100485)
+				(xy 175.825 104.955614) (xy 176.025 104.955614) (xy 176.423882 104.100485) (xy 175.925 103.491143)
+				(xy 175.426118 104.100485)
 			)
 		)
 	)
 	(zone
-		(net 2)
-		(net_name "+3V3")
+		(net 7)
+		(net_name "/vin")
 		(layer "F.Cu")
 		(name "$teardrop_padvia$")
 		(hatch none 0.1)
-		(priority 30008)
+		(priority 30000)
 		(attr
 			(teardrop
@@
 		(polygon
 			(pts
-				(xy 175.825 104.955614) (xy 176.025 104.955614) (xy 176.423882 104.100485) (xy 175.925 103.491143)
-				(xy 175.426118 104.100485)
+				(xy 189.38033 88.423883) (xy 189.733883 88.07033) (xy 188.849999 86.125786) (xy 187.499293 86.189293)
+				(xy 187.735785 87.839999)
 			)
 		)
@@
 		(net_name "+3V3")
 		(layer "F.Cu")
-		(hatch edge 0.5)
+		(name "$teardrop_padvia$")
+		(hatch none 0.1)
+		(priority 30005)
+		(attr
+			(teardrop
+				(type padvia)
+			)
+		)
 		(connect_pads yes
 			(clearance 0)
 		)
-		(min_thickness 0.25)
+		(min_thickness 0.0254)
 		(filled_areas_thickness no)
 		(fill yes
-			(mode hatch)
 			(thermal_gap 0.5)
 			(thermal_bridge_width 0.5)
-			(hatch_thickness 1)
-			(hatch_gap 1.5)
-			(hatch_orientation 0)
-			(hatch_border_algorithm hatch_thickness)
-			(hatch_min_hole_area 0.3)
+			(island_removal_mode 1)
+			(island_area_min 10)
 		)
 		(polygon
 			(pts
-				(xy 220.88 88.04) (xy 227.38 88.04) (xy 227.39 88.05) (xy 227.39 91.44) (xy 220.88 91.44)
+				(xy 175.040505 102.466227) (xy 174.899084 102.607648) (xy 175.325 103.740671) (xy 175.925707 103.49285)
+				(xy 175.910057 102.628672)
 			)
 		)
 	)
 	(zone
-		(net 2)
-		(net_name "+3V3")
+		(net 26)
+		(net_name "/io11")
 		(layer "F.Cu")
 		(name "$teardrop_padvia$")
 		(hatch none 0.1)
-		(priority 30009)
+		(priority 30010)
 		(attr
 			(teardrop
@@
 		(polygon
 			(pts
-				(xy 176.025 102.028672) (xy 175.825 102.028672) (xy 175.426118 102.883801) (xy 175.925 103.493143)
-				(xy 176.423882 102.883801)
+				(xy 171.825 104.955614) (xy 172.025 104.955614) (xy 172.423882 104.100485) (xy 171.925 103.491143)
+				(xy 171.426118 104.100485)
+			)
+		)
+	)
+	(zone
+		(net 2)
+		(net_name "+3V3")
+		(layer "F.Cu")
+		(hatch edge 0.5)
+		(connect_pads yes
+			(clearance 0)
+		)
+		(min_thickness 0.25)
+		(filled_areas_thickness no)
+		(fill yes
+			(mode hatch)
+			(thermal_gap 0.5)
+			(thermal_bridge_width 0.5)
+			(hatch_thickness 1)
+			(hatch_gap 1.5)
+			(hatch_orientation 0)
+			(hatch_border_algorithm hatch_thickness)
+			(hatch_min_hole_area 0.3)
+		)
+		(polygon
+			(pts
+				(xy 220.88 88.04) (xy 227.38 88.04) (xy 227.39 88.05) (xy 227.39 91.44) (xy 220.88 91.44)
 			)
 		)
@@
 			(thermal_gap 0.5)
 			(thermal_bridge_width 0.5)
-			(hatch_thickness 1)
-			(hatch_gap 1.5)
+			(hatch_thickness 3)
+			(hatch_gap 1)
 			(hatch_orientation 0)
 			(hatch_border_algorithm hatch_thickness)
@@
 		(polygon
 			(pts
-				(xy 180.97 89.51) (xy 180.97 92.47) (xy 182.5 92.47) (xy 182.5 89.51)
+				(xy 180.97 89.51) (xy 180.97 92.47) (xy 182.68 92.47) (xy 182.68 89.51)
 			)
 		)
@@
 		(polygon
 			(pts
-				(xy 168.71 89.6) (xy 168.71 83.09) (xy 184.06 83.09) (xy 184.06 89.6)
+				(xy 168.71 89.6) (xy 168.71 83.09) (xy 183.81 83.09) (xy 183.81 89.6)
 			)
 		)
