File: kicad/mdb-slave-esp32s3/mdb-slave-esp32s3.kicad_pcb (KiCad board)
At the start: 2 copper layers, 39 x 40 mm, 46 parts, among them J1 MDB_Connector, J2 USB_C_Receptacle_USB2.0_16P, J3 Conn_01x03_Pin, J8 Conn_01x04_Pin, Q7 MMBT3904, SW1 SW_Push, U1 TLP785, U3 ESP32-S3FH4R2, U4 TLP785, U5 LM2594HVM-3.3, Y1 Crystal_GND24

Commit message: routing...
Routing:
- net +3V3: track 120.2 -> 119.5 mm
Changed lines of the file:
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@@
+	)
+	(segment
+		(start 201.835025 104.824975)
+		(end 202.93 105.91995)
+		(width 0.2032)
+		(layer "F.Cu")
+		(net 2)
 	)
 	(segment
@@
 	)
 	(segment
-		(start 202.365025 106.3419)
-		(end 202.93 106.906875)
-		(width 0.2032)
-		(layer "F.Cu")
-		(net 2)
-	)
-	(segment
 		(start 182.803334 97.9925)
 		(end 182.8225 97.9925)
@@
 	)
 	(segment
+		(start 202.93 105.91995)
+		(end 202.93 106.906875)
+		(width 0.2032)
+		(layer "F.Cu")
+		(net 2)
+	)
+	(segment
 		(start 182.803334 97.9925)
 		(end 182.803334 96.466667)
@@
 		(end 178.995 97.955)
 		(width 0.2)
-		(layer "F.Cu")
-		(net 2)
-	)
-	(segment
-		(start 202.365025 105.354975)
-		(end 202.365025 106.3419)
-		(width 0.2032)
 		(layer "F.Cu")
 		(net 2)
@@
 	)
 	(via
-		(at 202.365025 105.354975)
+		(at 201.835025 104.824975)
 		(size 0.8)
 		(drill 0.4)
@@
 	)
 	(segment
-		(start 200.75005 103.74)
-		(end 202.365025 105.354975)
-		(width 0.508)
-		(layer "B.Cu")
-		(net 2)
-	)
-	(segment
 		(start 173.135 98.846667)
 		(end 173.361667 98.62)
@@
 	)
 	(segment
-		(start 202.365025 98.430025)
+		(start 200.75005 103.74)
+		(end 191.07 103.74)
+		(width 0.508)
+		(layer "B.Cu")
+		(net 2)
+	)
+	(segment
+		(start 201.835025 104.824975)
+		(end 200.75005 103.74)
+		(width 0.508)
+		(layer "B.Cu")
+		(net 2)
+	)
+	(segment
+		(start 201.835025 97.900025)
 		(end 201.815 97.88)
 		(width 0.2032)
-		(layer "B.Cu")
-		(net 2)
-	)
-	(segment
-		(start 191.07 103.74)
-		(end 200.75005 103.74)
-		(width 0.508)
 		(layer "B.Cu")
 		(net 2)
@@
 	)
 	(segment
-		(start 202.365025 105.354975)
-		(end 202.365025 98.430025)
-		(width 0.2032)
-		(layer "B.Cu")
-		(net 2)
-	)
-	(segment
 		(start 191.07 103.02)
 		(end 187.53 99.48)
@@
 		(end 186.67 98.62)
 		(width 0.508)
+		(layer "B.Cu")
+		(net 2)
+	)
+	(segment
+		(start 201.835025 104.824975)
+		(end 201.835025 97.900025)
+		(width 0.2032)
 		(layer "B.Cu")
 		(net 2)
@@
 	)
 	(segment
-		(start 203.6 91.765)
-		(end 205.8274 93.9924)
-		(width 0.508)
-		(layer "F.Cu")
-		(net 7)
-	)
-	(segment
 		(start 187.925 85.99)
 		(end 190.185 88.25)
@@
 	)
 	(segment
-		(start 205.8274 93.9924)
+		(start 205.8274 94.8874)
 		(end 205.8274 112.5976)
+		(width 0.508)
+		(layer "F.Cu")
+		(net 7)
+	)
+	(segment
+		(start 203.6 91.765)
+		(end 203.6 92.66)
+		(width 0.508)
+		(layer "F.Cu")
+		(net 7)
+	)
+	(segment
+		(start 203.6 92.66)
+		(end 205.8274 94.8874)
 		(width 0.508)
 		(layer "F.Cu")
@@
 	)
 	(zone
-		(net 27)
-		(net_name "/io11")
+		(net 3)
+		(net_name "GND")
 		(layer "F.Cu")
 		(name "$teardrop_padvia$")
 		(hatch none 0.1)
-		(priority 30009)
+		(priority 30005)
 		(attr
 			(teardrop
@@
 		(polygon
 			(pts
-				(xy 174.598471 94.946667) (xy 174.598471 94.746667) (xy 173.743342 94.347785) (xy 173.134 94.846667)
-				(xy 173.743342 95.345549)
+				(xy 174.61 100.948267) (xy 174.61 100.745067) (xy 173.855671 100.265697) (xy 173.134 100.846667)
+				(xy 173.855671 101.427637)
 			)
 		)
@@
 		(name "$teardrop_padvia$")
 		(hatch none 0.1)
-		(priority 30012)
+		(priority 30010)
 		(attr
 			(teardrop
@@
 		(polygon
 			(pts
-				(xy 180.267289 115.084605) (xy 180.123605 115.228289) (xy 180.549 116.217106) (xy 181.049707 116.010707)
-				(xy 180.78476 115.038654)
+				(xy 182.007579 115.664) (xy 182.007579 115.156) (xy 181.4509 115.16838) (xy 181.048 116.01) (xy 181.549 116.286434)
 			)
 		)
 	)
 	(zone
-		(net 11)
-		(net_name "/mdb_communications_common")
+		(net 3)
+		(net_name "GND")
 		(layer "F.Cu")
 		(name "$teardrop_padvia$")
 		(hatch none 0.1)
-		(priority 30000)
+		(priority 30012)
 		(attr
 			(teardrop
@@
 		(polygon
 			(pts
-				(xy 198.051017 93.357438) (xy 198.192438 93.216017) (xy 197.675 91.425786) (xy 196.324293 91.489293)
-				(xy 196.539087 93.118301)
+				(xy 180.267289 115.084605) (xy 180.123605 115.228289) (xy 180.549 116.217106) (xy 181.049707 116.010707)
+				(xy 180.78476 115.038654)
 			)
 		)
@@
 		(name "$teardrop_padvia$")
 		(hatch none 0.1)
-		(priority 30010)
+		(priority 30011)
 		(attr
 			(teardrop
@@
 		(polygon
 			(pts
-				(xy 182.007579 115.664) (xy 182.007579 115.156) (xy 181.4509 115.16838) (xy 181.048 116.01) (xy 181.549 116.286434)
+				(xy 188.730421 115.156) (xy 188.730421 115.664) (xy 189.189 116.286434) (xy 189.69 116.01) (xy 189.287099 115.16838)
 			)
 		)
 	)
 	(zone
-		(net 10)
-		(net_name "/mdb_master_transmit")
+		(net 11)
+		(net_name "/mdb_communications_common")
 		(layer "F.Cu")
 		(name "$teardrop_padvia$")
 		(hatch none 0.1)
-		(priority 30002)
+		(priority 30000)
 		(attr
 			(teardrop
@@
 		(polygon
 			(pts
-				(xy 194.103805 92.667489) (xy 194.247489 92.523805) (xy 193.467635 91.077629) (xy 192.124293 91.489293)
-				(xy 192.760517 92.968593)
+				(xy 198.051017 93.357438) (xy 198.192438 93.216017) (xy 197.675 91.425786) (xy 196.324293 91.489293)
+				(xy 196.539087 93.118301)
 			)
 		)
 	)
 	(zone
-		(net 3)
-		(net_name "GND")
+		(net 23)
+		(net_name "/io10")
 		(layer "F.Cu")
 		(name "$teardrop_padvia$")
 		(hatch none 0.1)
-		(priority 30005)
+		(priority 30008)
 		(attr
 			(teardrop
@@
 		(polygon
 			(pts
-				(xy 174.61 100.948267) (xy 174.61 100.745067) (xy 173.855671 100.265697) (xy 173.134 100.846667)
-				(xy 173.855671 101.427637)
+				(xy 174.598471 96.946667) (xy 174.598471 96.746667) (xy 173.743342 96.347785) (xy 173.134 96.846667)
+				(xy 173.743342 97.345549)
 			)
 		)
 	)
 	(zone
-		(net 3)
-		(net_name "GND")
+		(net 10)
+		(net_name "/mdb_master_transmit")
 		(layer "F.Cu")
 		(name "$teardrop_padvia$")
 		(hatch none 0.1)
-		(priority 30013)
+		(priority 30002)
 		(attr
 			(teardrop
@@
 		(polygon
 			(pts
-				(xy 180.192157 120.9234) (xy 180.192157 121.1266) (xy 180.872955 121.067877) (xy 181.05 120.21)
-				(xy 180.549 119.996303)
+				(xy 194.103805 92.667489) (xy 194.247489 92.523805) (xy 193.467635 91.077629) (xy 192.124293 91.489293)
+				(xy 192.760517 92.968593)
 			)
 		)
 	)
 	(zone
-		(net 23)
-		(net_name "/io10")
+		(net 3)
+		(net_name "GND")
 		(layer "F.Cu")
 		(name "$teardrop_padvia$")
 		(hatch none 0.1)
-		(priority 30008)
+		(priority 30013)
 		(attr
 			(teardrop
@@
 		(polygon
 			(pts
-				(xy 174.598471 96.946667) (xy 174.598471 96.746667) (xy 173.743342 96.347785) (xy 173.134 96.846667)
-				(xy 173.743342 97.345549)
+				(xy 180.192157 120.9234) (xy 180.192157 121.1266) (xy 180.872955 121.067877) (xy 181.05 120.21)
+				(xy 180.549 119.996303)
 			)
 		)
 	)
 	(zone
-		(net 3)
-		(net_name "GND")
+		(net 2)
+		(net_name "+3V3")
 		(layer "F.Cu")
 		(name "$teardrop_padvia$")
 		(hatch none 0.1)
-		(priority 30011)
+		(priority 30007)
 		(attr
 			(teardrop
@@
 		(polygon
 			(pts
-				(xy 188.730421 115.156) (xy 188.730421 115.664) (xy 189.189 116.286434) (xy 189.69 116.01) (xy 189.287099 115.16838)
+				(xy 174.598471 98.946667) (xy 174.598471 98.746667) (xy 173.743342 98.347785) (xy 173.134 98.846667)
+				(xy 173.743342 99.345549)
 			)
 		)
 	)
 	(zone
-		(net 12)
-		(net_name "/mdb_master_receive")
+		(net 27)
+		(net_name "/io11")
 		(layer "F.Cu")
 		(name "$teardrop_padvia$")
 		(hatch none 0.1)
-		(priority 30001)
+		(priority 30009)
 		(attr
 			(teardrop
@@
 		(polygon
 			(pts
-				(xy 189.792438 89.763983) (xy 189.651017 89.622562) (xy 188.139088 89.861698) (xy 187.924293 91.490707)
-				(xy 189.275 91.554214)
+				(xy 174.598471 94.946667) (xy 174.598471 94.746667) (xy 173.743342 94.347785) (xy 173.134 94.846667)
+				(xy 173.743342 95.345549)
 			)
 		)
 	)
 	(zone
-		(net 27)
-		(net_name "/io11")
+		(net 23)
+		(net_name "/io10")
 		(layer "F.Cu")
 		(name "$teardrop_padvia$")
 		(hatch none 0.1)
-		(priority 30006)
+		(priority 30004)
 		(attr
 			(teardrop
@@
 		(polygon
 			(pts
-				(xy 172.109084 95.731162) (xy 172.250505 95.872583) (xy 173.383528 95.446667) (xy 173.135707 94.84596)
-				(xy 172.271529 94.861609)
+				(xy 171.92558 97.592999) (xy 172.067001 97.73442) (xy 173.327746 97.446667) (xy 173.135707 96.84596)
+				(xy 172.271529 96.729613)
 			)
 		)
 	)
 	(zone
-		(net 23)
-		(net_name "/io10")
+		(net 27)
+		(net_name "/io11")
 		(layer "F.Cu")
 		(name "$teardrop_padvia$")
 		(hatch none 0.1)
-		(priority 30004)
+		(priority 30006)
 		(attr
 			(teardrop
@@
 		(polygon
 			(pts
-				(xy 171.92558 97.592999) (xy 172.067001 97.73442) (xy 173.327746 97.446667) (xy 173.135707 96.84596)
-				(xy 172.271529 96.729613)
+				(xy 172.109084 95.731162) (xy 172.250505 95.872583) (xy 173.383528 95.446667) (xy 173.135707 94.84596)
+				(xy 172.271529 94.861609)
 			)
 		)
 	)
 	(zone
-		(net 2)
-		(net_name "+3V3")
+		(net 12)
+		(net_name "/mdb_master_receive")
 		(layer "F.Cu")
 		(name "$teardrop_padvia$")
 		(hatch none 0.1)
-		(priority 30007)
+		(priority 30001)
 		(attr
 			(teardrop
@@
 		(polygon
 			(pts
-				(xy 174.598471 98.946667) (xy 174.598471 98.746667) (xy 173.743342 98.347785) (xy 173.134 98.846667)
-				(xy 173.743342 99.345549)
-			)
-		)
+				(xy 189.792438 89.763983) (xy 189.651017 89.622562) (xy 188.139088 89.861698) (xy 187.924293 91.490707)
+				(xy 189.275 91.554214)
+			)
+		)
