File: kicad/mdb-slave-esp32s3/mdb-slave-esp32s3.kicad_sch (KiCad schematic)
At the start: 47 parts, among them J1 MDB_Connector, J2 USB_C_Receptacle_USB2.0_16P, J3 Conn_01x03_Pin, J8 Conn_01x04_Pin, Q7 MMBT3904, SW1 SW_Push, U1 TLP785, U3 ESP32-S3FH4R2, U4 TLP785, U5 LM2594HVM-3.3, Y1 Crystal_GND24

Commit message: Update KiCad PCB and schematic files
Co-Authored-By: Claude Sonnet 4.6 <noreply@anthropic.com>
Parts:
- removed R11: 1k, Resistor_SMD:R_0603_1608Metric, symbol Device:R
- removed R15: 10k, Resistor_SMD:R_0603_1608Metric, symbol Device:R
- removed TH1: Thermistor_NTC, Resistor_SMD:R_0603_1608Metric, symbol Device:Thermistor_NTC
- added R1: 4K7, Resistor_SMD:R_0603_1608Metric, symbol Device:R
Connections:
- net io13: now also R1.1
- net at Q7.1 (B): now also R1.2

Commit message: chore(kicad): update schematic and PCB layouts
Co-Authored-By: Claude Opus 4.7 <noreply@anthropic.com>
Parts:
- added C7: 0.1uF, Capacitor_SMD:C_0603_1608Metric, symbol Device:C
Connections:
- net +3V3: now also C7.2
- net GND: now also C7.1
Other:
- moved on the sheet: D2, J1, J3, J8, Q7, R1, R10, R13, R2, R24, R25, R5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
