File: kicad/mdb-slave-esp32s3/mdb-slave-esp32s3.kicad_sch (KiCad schematic)
At the start: 46 parts, among them J1 MDB_Connector, J2 USB_C_Receptacle_USB2.0_16P, J3 Conn_01x03_Pin, J8 Conn_01x04_Pin, Q7 MMBT3904, SW1 SW_Push, U1 TLP785, U3 ESP32-S3FH4R2, U4 TLP785, U5 LM2594HVM-3.3, Y1 Crystal_GND24

Commit message: tlp185 to tlp785
Parts:
- U1, U4: LCSC# C128776 -> C45445
Changed lines of the file:
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@@
 			)
 		)
-		(property "LCSC#" "C128776"
+		(property "LCSC#" "C45445"
 			(at 358.14 88.9 0)
 			(effects
@@
 			)
 		)
-		(property "LCSC#" "C128776"
+		(property "LCSC#" "C45445"
 			(at 358.14 104.14 0)
 			(effects
