File: kicad/mdb-slave-esp32s3/mdb-slave-esp32s3.kicad_sch (KiCad schematic)
At the start: 46 parts, among them J1 MDB_Connector, J2 USB_C_Receptacle_USB2.0_16P, J3 Conn_01x03_Pin, J8 Conn_01x04_Pin, Q7 MMBT3904, SW1 SW_Push, U1 TLP785, U3 ESP32-S3FH4R2, U4 TLP785, U5 LM2594HVM-3.3, Y1 Crystal_GND24

Commit message: fix(hardware): standardize Value field notation in schematics
4K7→4.7k, 22ohm→22R, 470ohm→470R, 1.8pf→1.8pF, 2.4nh→2.4nH,
5.6nh→5.6nH, 3.9nh→3.9nH, Crystal_GND24→40MHz, FerriteBead_Small→FerriteBead

Co-Authored-By: Claude Sonnet 4.6 <noreply@anthropic.com>
Parts:
- C4: value 1.8pf -> 1.8pF
- FB2: value FerriteBead_Small -> FerriteBead
- L1: value 2.4nh -> 2.4nH
- R1, R24, R25: value 4K7 -> 4.7k
- R2, R5: value 470ohm -> 470R
- Y1: value Crystal_GND24 -> 40MHz
Changed lines of the file:
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@@
 			)
 		)
-		(property "Value" "4K7"
+		(property "Value" "4.7k"
 			(at 256.54 52.0699 0)
 			(effects
@@
 			)
 		)
-		(property "Value" "4K7"
+		(property "Value" "4.7k"
 			(at 256.54 96.52 90)
 			(effects
@@
 			)
 		)
-		(property "Value" "4K7"
+		(property "Value" "4.7k"
 			(at 269.24 49.5299 0)
 			(effects
@@
 			)
 		)
-		(property "Value" "470ohm"
+		(property "Value" "470R"
 			(at 373.38 111.7599 0)
 			(effects
@@
 			)
 		)
-		(property "Value" "FerriteBead_Small"
+		(property "Value" "FerriteBead"
 			(at 137.1219 26.67 90)
 			(effects
@@
 			)
 		)
-		(property "Value" "Crystal_GND24"
+		(property "Value" "40MHz"
 			(at 86.36 132.2068 90)
 			(effects
@@
 			)
 		)
-		(property "Value" "470ohm"
+		(property "Value" "470R"
 			(at 345.44 82.55 90)
 			(effects
@@
 			)
 		)
-		(property "Value" "1.8pf"
+		(property "Value" "1.8pF"
 			(at 35.56 106.68 90)
 			(effects
@@
 			)
 		)
-		(property "Value" "2.4nh"
+		(property "Value" "2.4nH"
 			(at 30.48 119.38 0)
 			(effects

Commit message: fix(kicad): resolve ERC violations in mdb-slave-esp32s3 schematics
All ERC validations pass now on both sim7080g and base variants.

Co-Authored-By: Claude Sonnet 5 <noreply@anthropic.com>
Connections:
- net io1: no longer names the net of U3.6 (GPIO1/ADC1_CH0)
- net io12: no longer names the net of U3.17 (GPIO12/ADC2_CH1)
- net io14: no longer names the net of U3.19 (GPIO14/ADC2_CH3)
- net io17: no longer names the net of U3.23 (GPIO17/ADC2_CH6)
- net io18: no longer names the net of U3.24 (GPIO18/ADC2_CH7)
- net io2: no longer names the net of U3.7 (GPIO2/ADC1_CH1)
- net io7: no longer names the net of U3.12 (GPIO7/ADC1_CH6)
- net io8: no longer names the net of U3.13 (GPIO8/ADC1_CH7)
- net io9: no longer names the net of U3.14 (GPIO9/ADC1_CH8)
- net u0rxd: no longer names the net of U3.50 (U0RXD/PROG/GPIO44)
- net u0txd: no longer names the net of U3.49 (U0TXD/PROG/GPIO43)
- no-connect marks 30 -> 41
