File: kicad/mdb-dual-esp32s3-sim7080g/mdb-dual-esp32s3-sim7080g.kicad_pcb (KiCad board)
At the start: 2 copper layers, 65 x 40 mm, 82 parts, among them J1 USB_C_Receptacle_USB2.0_16P, J2 JAE_SIM_Card_SF72S006, J3 Conn_01x03_Pin, J4 Conn_Coaxial, J5 Conn_Coaxial, J6 MDB_Connector, J7 Conn_01x03_Pin, J8 Conn_01x04_Pin, Q1 MMBT3904, Q2 MMBT3904, Q3 MMBT3904, Q4 MMBT3904, Q5 MMBT3904, Q6 MMBT3904, Q7 MMBT3904, SW1 SW_Push, U1 ESP32-S3FH4R2, U2 SIM7080G, U3 LM2594HVM-3.3, U4 TLP785, U5 TLP785, Y1 Crystal_GND24

Commit message: routing...
Parts:
- removed AE1: Antenna, RF_Antenna:Texas_SWRA117D_2.4GHz_Left
- removed D3: D_Schottky, Diode_SMD:D_SOD-123
- removed J3, J7: Conn_01x03_Pin, Connector_JST:JST_PH_B3B-PH-K_1x03_P2.00mm_Vertical
- removed Q5, Q6, Q7: MMBT3904, Package_TO_SOT_SMD:SOT-23
- removed R15, R21, R23: 4K7, Resistor_SMD:R_0603_1608Metric
- removed R20, R22, R27: 10k, Resistor_SMD:R_0603_1608Metric
- removed REF**: OSHW-Logo_11.4x12mm_SilkScreen, Symbol:OSHW-Logo_11.4x12mm_SilkScreen
- added C18: 22pF, Capacitor_SMD:C_0603_1608Metric, F.Cu at (168.4, 107.4)
- added C22: 22pF, Capacitor_SMD:C_0603_1608Metric, F.Cu at (171.8, 107.4)
- added D5: D_Schottky, Diode_SMD:D_SOD-123, F.Cu at (177.9, 107.5)
- added J10: Conn_Coaxial, Connector_Coaxial:U.FL_Hirose_U.FL-R-SMT-1_Vertical, F.Cu at (178.3, 98.4)
- added J9: MDB_Connector, Connector_Molex:Molex_Mini-Fit_Jr_5566-06A_2x03_P4.20mm_Vertical, F.Cu at (170.4, 86.2)
- added L5: 4.7uF, Inductor_SMD:L_APV_ANR3015, F.Cu at (173.3, 104.1)
- added Q8: MMBT3904, Package_TO_SOT_SMD:SOT-23, F.Cu at (173.1, 98.8)
- added R26: 15k, Resistor_SMD:R_0603_1608Metric, F.Cu at (179.5, 110.5)
- added R28: 110k, Resistor_SMD:R_0603_1608Metric, F.Cu at (168.3, 97.3)
- added R30: 10k, Resistor_SMD:R_0603_1608Metric, F.Cu at (168.3, 99.8)
- added R31: 4K7, Resistor_SMD:R_0603_1608Metric, F.Cu at (168.3, 102.3)
- added R32: 1k, Resistor_SMD:R_0603_1608Metric, F.Cu at (168.3, 104.8)
- added U7: MT3608, Package_TO_SOT_SMD:SOT-23-6, F.Cu at (178.2, 104.2)
- moved L1 14.1 mm to (191.1, 101.4)
- moved C1 14.1 mm to (191.1, 103.0)
- moved J8 9.14 mm to (175.2, 112.2)
- moved R25 9.14 mm to (168.2, 115.6)
- moved R24 9.14 mm to (171.4, 115.6)
- moved C3 2.53 mm to (182.5, 96.6)
- moved C9 2.53 mm to (184.9, 100.8)
- moved FB1 2.53 mm to (183.3, 100.8)
- moved R1 2.53 mm to (182.5, 98.3)
- moved R8 2.53 mm to (181.7, 100.8)
- moved SW1 2.25 mm to (171.7, 120.4)
- moved U1 1.42 mm to (186.6, 107.4)
Routing:
- net +3V3: track 217.8 -> 0.00 mm, vias 8 -> 0
- net GND: track 180.7 -> 0.00 mm, vias 30 -> 0
- net /vin: track 80.9 -> 0.00 mm, vias 1 -> 0
- net /io14: track 53.6 -> 0.00 mm, vias 2 -> 0
- net /boot: track 51.0 -> 0.00 mm
- net /io18: track 41.7 -> 0.00 mm, vias 2 -> 0
- net /io21: track 34.1 -> 0.00 mm, vias 2 -> 0
- net /io12: track 32.1 -> 0.00 mm, vias 2 -> 0
- net /io17: track 30.2 -> 0.00 mm, vias 2 -> 0
- net /mdb_communications_common: track 27.8 -> 0.00 mm
- net /io4: track 26.8 -> 0.00 mm, vias 2 -> 0
- net /mdb_master_receive: track 25.2 -> 0.00 mm
- net /mdb_master_transmit: track 21.0 -> 0.00 mm
- net /sim_vdd_ext: track 20.5 -> 0.00 mm, vias 2 -> 0
- net Net-(J2-CLK): track 20.4 -> 0.00 mm
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Other:
- board size 65 x 40 mm -> 67.4 x 40 mm
- board text removed: "3v3"
- board text removed: "gnd"
- board text removed: "pulse"
- board text removed: "rx"
- board text removed: "scl"
- board text removed: "sda"
- board text removed: "tx"
- board text removed: "vin"
