File: kicad/mdb-dual-esp32s3-sim7080g/mdb-dual-esp32s3-sim7080g.kicad_sch (KiCad schematic)
At the start: 99 parts, among them J1 USB_C_Receptacle_USB2.0_16P, J2 JAE_SIM_Card_SF72S006, J3 Conn_01x03_Pin, J4 Conn_Coaxial, J5 Conn_Coaxial, J6 MDB_Connector, J7 Conn_01x03_Pin, J8 Conn_01x04_Pin, J9 MDB_Connector, Q1 MMBT3904, Q2 MMBT3904, Q3 MMBT3904, Q4 MMBT3904, Q5 MMBT3904, Q6 MMBT3904, Q7 MMBT3904, Q8 MMBT3904, SW1 SW_Push, U1 ESP32-S3FH4R2, U2 SIM7080G, U3 LM2594HVM-3.3, U4 TLP785, U5 TLP785, U7 MT3608, U8 MAX3232, Y1 Crystal_GND24

Commit message: routing...
Parts:
- removed AE1: Antenna, RF_Antenna:Texas_SWRA117D_2.4GHz_Left, symbol Device:Antenna
- removed C23, C24, C25, C26, C27: 0.1uF, Capacitor_SMD:C_0603_1608Metric, symbol Device:C
- removed D3: D_Schottky, Diode_SMD:D_SOD-123, symbol Device:D_Schottky
- removed J3, J7: Conn_01x03_Pin, Connector_JST:JST_PH_B3B-PH-K_1x03_P2.00mm_Vertical, symbol Connector:Conn_01x03_Pin
- removed Q5, Q6, Q7: MMBT3904, Package_TO_SOT_SMD:SOT-23, symbol Transistor_BJT:MMBT3904
- removed R15, R21, R23: 4K7, Resistor_SMD:R_0603_1608Metric, symbol Device:R
- removed R20, R22, R27: 10k, Resistor_SMD:R_0603_1608Metric, symbol Device:R
- removed U8: MAX3232, Package_SO:SOIC-16_3.9x9.9mm_P1.27mm, symbol Interface_UART:MAX3232
- added J10: Conn_Coaxial, Connector_Coaxial:U.FL_Hirose_U.FL-R-SMT-1_Vertical, symbol Connector:Conn_Coaxial
Connections:
- net GND: now also J10.2 (Ext)
- net at C1.1, L1.2: now also J10.1 (In)
- net mdb_target_receive renamed mdb_master_receive
- net mdb_target_transmit renamed mdb_master_transmit
Other:
- moved on the sheet: BZ1, C1, C10, C11, C12, C13, C14, C15, C16, C17, C18, C19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
