File: kicad/mdb-dual-esp32s3/mdb-dual-esp32s3.kicad_pcb (KiCad board)
At the start: 2 copper layers, 39 x 40 mm, 52 parts, among them J1 MDB_Connector, J2 USB_C_Receptacle_USB2.0_16P, J4 Conn_Coaxial, J8 Conn_01x04_Pin, J9 MDB_Connector, Q8 MMBT3904, SW1 SW_Push, U1 TLP785, U3 ESP32-S3FH4R2, U4 TLP785, U5 LM2594HVM-3.3, U7 MT3608, Y1 Crystal_GND24

Commit message: routing
Parts:
- added C7: 0.1uF, Capacitor_SMD:C_0603_1608Metric, F.Cu at (176.8, 114.2)
- moved C18 11.2 mm to (183.2, 96.1), turned to 0 degrees
- moved FB2 0.10 mm to (183.2, 97.6)
- moved C14 0.05 mm to (183.2, 99.2)
Routing:
- net GND: track 48.5 -> 51.1 mm
- net +3V3: track 155.3 -> 157.4 mm
- net /io11: track 26.3 -> 27.2 mm
- net /io21: track 29.1 -> 28.6 mm

Commit message: routing...
Parts:
- removed R30: 10k, Resistor_SMD:R_0603_1608Metric
- added R1: 1k, Resistor_SMD:R_0603_1608Metric, F.Cu at (173.9, 103.9)
- moved R31 3.26 mm to (173.9, 100.7), turned to 0 degrees
Connections:
- R31 pad 1: /io2 -> /mdb_controller_transmit
- R31 pad 2: Net-(Q8-B) -> +5V
Other:
- board text added: "3v3"
- board text added: "gnd"
- board text added: "io10"
- board text added: "io11"
- board text removed: "gnd,3v3,io10,io11"
