File: kicad/mdb-dual-esp32s3/mdb-dual-esp32s3.kicad_sch (KiCad schematic)
At the start: 52 parts, among them J1 MDB_Connector, J2 USB_C_Receptacle_USB2.0_16P, J4 Conn_Coaxial, J8 Conn_01x04_Pin, J9 MDB_Connector, Q8 MMBT3904, SW1 SW_Push, U1 TLP785, U3 ESP32-S3FH4R2, U4 TLP785, U5 LM2594HVM-3.3, U7 MT3608, Y1 Crystal_GND24

Commit message: routing
Parts:
- added C7: 0.1uF, Capacitor_SMD:C_0603_1608Metric, symbol Device:C
Connections:
- net +3V3: now also C7.1
- net GND: now also C7.2
Other:
- moved on the sheet: J8, R24, R25

Commit message: routing...
Parts:
- removed R30: 10k, Resistor_SMD:R_0603_1608Metric, symbol Device:R
- added R1: 1k, Resistor_SMD:R_0603_1608Metric, symbol Device:R
Connections:
- net +5V: now also R31.2
- net io2: now also R1.2; no longer R31.1
- net mdb_controller_transmit: now also R31.1
- net at Q8.1 (B): now also R1.1; no longer R31.2
Other:
- moved on the sheet: R31, R32
Changed lines of the file:
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@@
 	)
 	(junction
-		(at 285.75 93.98)
+		(at 280.67 93.98)
 		(diameter 0)
 		(color 0 0 0 0)
@@
 	)
 	(junction
-		(at 229.87 68.58)
-		(diameter 0)
-		(color 0 0 0 0)
-	)
-	(junction
 		(at 241.3 167.64)
 		(diameter 0)
@@
 	)
 	(junction
+		(at 229.87 68.58)
+		(diameter 0)
+		(color 0 0 0 0)
+	)
+	(junction
 		(at 124.46 102.87)
 		(diameter 0)
@@
 	(wire
 		(pts
-			(xy 285.75 88.9) (xy 285.75 93.98)
+			(xy 280.67 88.9) (xy 280.67 93.98)
 		)
 		(stroke
@@
 	(wire
 		(pts
-			(xy 279.4 93.98) (xy 285.75 93.98)
+			(xy 274.32 93.98) (xy 280.67 93.98)
 		)
 		(stroke
@@
 	(wire
 		(pts
-			(xy 285.75 110.49) (xy 285.75 105.41)
+			(xy 280.67 110.49) (xy 280.67 105.41)
 		)
 		(stroke
@@
 	(wire
 		(pts
-			(xy 285.75 93.98) (xy 285.75 97.79)
+			(xy 280.67 93.98) (xy 280.67 97.79)
 		)
 		(stroke
@@
 	)
 	(label "io1"
-		(at 285.75 88.9 0)
+		(at 280.67 88.9 0)
 		(effects
 			(font
@@
 	)
 	(label "mdb_controller_receive"
-		(at 279.4 93.98 180)
+		(at 274.32 93.98 180)
 		(effects
 			(font
@@
 	(symbol
 		(lib_id "Device:R")
-		(at 226.06 68.58 270)
-		(unit 1)
-		(exclude_from_sim no)
-		(in_bom yes)
-		(on_board yes)
-		(dnp no)
-		(fields_autoplaced yes)
-		(property "Reference" "R30"
-			(at 226.06 62.23 90)
-			(effects
-				(font
-					(size 1.27 1.27)
-				)
-			)
-		)
-		(property "Value" "10k"
-			(at 226.06 64.77 90)
-			(effects
-				(font
-					(size 1.27 1.27)
-				)
-			)
-		)
-		(property "Footprint" "Resistor_SMD:R_0603_1608Metric"
-			(at 226.06 66.802 90)
-			(effects
-				(font
-					(size 1.27 1.27)
-				)
-				(hide yes)
-			)
-		)
-		(property "Datasheet" "~"
-			(at 226.06 68.58 0)
-			(effects
-				(font
-					(size 1.27 1.27)
-				)
-				(hide yes)
-			)
-		)
-		(property "Description" ""
-			(at 226.06 68.58 0)
-			(effects
-				(font
-					(size 1.27 1.27)
-				)
-				(hide yes)
-			)
-		)
-		(property "LCSC#" "C98220"
-			(at 226.06 68.58 90)
-			(effects
-				(font
-					(size 1.27 1.27)
-				)
-				(hide yes)
-			)
-		)
-		(property "Sim.Device" ""
-			(at 226.06 68.58 90)
-			(effects
-				(font
-					(size 1.27 1.27)
-				)
-				(hide yes)
-			)
-		)
-		(property "Sim.Pins" ""
-			(at 226.06 68.58 90)
-			(effects
-				(font
-					(size 1.27 1.27)
-				)
-				(hide yes)
-			)
-		)
-		(property "Sim.Type" ""
-			(at 226.06 68.58 90)
-			(effects
-				(font
-					(size 1.27 1.27)
-				)
-				(hide yes)
-			)
-		)
-		(pin "1"
-		)
-		(pin "2"
-		)
-		(instances
-			(project "mdb-slave-esp32s3"
-				(path "/95980b25-0707-441d-ba83-7f6c6e1d1aaa"
-					(reference "R30")
-					(unit 1)
-				)
-			)
-		)
-	)
-	(symbol
-		(lib_id "Device:R")
 		(at 64.77 72.39 0)
 		(unit 1)
@@
 	)
 	(symbol
+		(lib_id "Device:R")
+		(at 236.22 81.28 0)
+		(unit 1)
+		(exclude_from_sim no)
+		(in_bom yes)
+		(on_board yes)
+		(dnp no)
+		(fields_autoplaced yes)
+		(property "Reference" "R1"
+			(at 238.76 80.0099 0)
+			(effects
+				(font
+					(size 1.27 1.27)
+				)
+				(justify left)
+			)
+		)
+		(property "Value" "1k"
+			(at 238.76 82.5499 0)
+			(effects
+				(font
+					(size 1.27 1.27)
+				)
+				(justify left)
+			)
+		)
+		(property "Footprint" "Resistor_SMD:R_0603_1608Metric"
+			(at 234.442 81.28 90)
+			(effects
+				(font
+					(size 1.27 1.27)
+				)
+				(hide yes)
+			)
+		)
+		(property "Datasheet" "~"
+			(at 236.22 81.28 0)
+			(effects
+				(font
+					(size 1.27 1.27)
+				)
+				(hide yes)
+			)
+		)
+		(property "Description" ""
+			(at 236.22 81.28 0)
+			(effects
+				(font
+					(size 1.27 1.27)
+				)
+				(hide yes)
+			)
+		)
+		(property "LCSC#" "C2907113"
+			(at 236.22 81.28 90)
+			(effects
+				(font
+					(size 1.27 1.27)
+				)
+				(hide yes)
+			)
+		)
+		(pin "1"
+		)
+		(pin "2"
+		)
+		(instances
+			(project "mdb-dual-esp32s3"
+				(path "/95980b25-0707-441d-ba83-7f6c6e1d1aaa"
+					(reference "R1")
+					(unit 1)
+				)
+			)
+		)
+	)
+	(symbol
 		(lib_id "Connector:Conn_Coaxial")
 		(at 29.21 99.06 90)
@@
 	(symbol
 		(lib_id "power:+3V3")
-		(at 285.75 110.49 180)
+		(at 280.67 110.49 180)
 		(unit 1)
 		(exclude_from_sim no)
@@
 		(fields_autoplaced yes)
 		(property "Reference" "#PWR067"
-			(at 285.75 106.68 0)
+			(at 280.67 106.68 0)
 			(effects
 				(font
@@
 		)
 		(property "Value" "+3V3"
-			(at 285.75 115.57 0)
+			(at 280.67 115.57 0)
 			(effects
 				(font
@@
 		)
 		(property "Footprint" ""
-			(at 285.75 110.49 0)
+			(at 280.67 110.49 0)
 			(effects
 				(font
@@
 		)
 		(property "Datasheet" ""
-			(at 285.75 110.49 0)
+			(at 280.67 110.49 0)
 			(effects
 				(font
@@
 		)
 		(property "Description" ""
-			(at 285.75 110.49 0)
+			(at 280.67 110.49 0)
 			(effects
 				(font
@@
 	(symbol
 		(lib_id "Device:R")
-		(at 236.22 81.28 180)
+		(at 226.06 68.58 270)
 		(unit 1)
 		(exclude_from_sim no)
@@
 		(fields_autoplaced yes)
 		(property "Reference" "R31"
-			(at 238.76 80.0099 0)
+			(at 226.06 62.23 90)
 			(effects
 				(font
 					(size 1.27 1.27)
 				)
-				(justify right)
 			)
 		)
 		(property "Value" "4K7"
-			(at 238.76 82.5499 0)
+			(at 226.06 64.77 90)
 			(effects
 				(font
 					(size 1.27 1.27)
 				)
-				(justify right)
 			)
 		)
 		(property "Footprint" "Resistor_SMD:R_0603_1608Metric"
-			(at 237.998 81.28 90)
+			(at 226.06 66.802 90)
 			(effects
 				(font
@@
 		)
 		(property "Datasheet" "~"
-			(at 236.22 81.28 0)
+			(at 226.06 68.58 0)
 			(effects
 				(font
@@
 		)
 		(property "Description" ""
-			(at 236.22 81.28 0)
+			(at 226.06 68.58 0)
 			(effects
 				(font
@@
 		)
 		(property "LCSC#" "C23162"
-			(at 236.22 81.28 0)
+			(at 226.06 68.58 0)
 			(effects
 				(font
@@
 		)
 		(property "Sim.Device" ""
-			(at 236.22 81.28 0)
+			(at 226.06 68.58 0)
 			(effects
 				(font
@@
 		)
 		(property "Sim.Pins" ""
-			(at 236.22 81.28 0)
+			(at 226.06 68.58 0)
 			(effects
 				(font
@@
 		)
 		(property "Sim.Type" ""
-			(at 236.22 81.28 0)
+			(at 226.06 68.58 0)
 			(effects
 				(font
@@
 	(symbol
 		(lib_id "Device:R")
-		(at 285.75 101.6 0)
+		(at 280.67 101.6 0)
 		(unit 1)
 		(exclude_from_sim no)
@@
 		(fields_autoplaced yes)
 		(property "Reference" "R32"
-			(at 288.29 100.3299 0)
+			(at 283.21 100.3299 0)
 			(effects
 				(font
@@
 		)
 		(property "Value" "1k"
-			(at 288.29 102.8699 0)
+			(at 283.21 102.8699 0)
 			(effects
 				(font
@@
 		)
 		(property "Footprint" "Resistor_SMD:R_0603_1608Metric"
-			(at 283.972 101.6 90)
+			(at 278.892 101.6 90)
 			(effects
 				(font
@@
 		)
 		(property "Datasheet" "~"
-			(at 285.75 101.6 0)
+			(at 280.67 101.6 0)
 			(effects
 				(font
@@
 		)
 		(property "Description" ""
-			(at 285.75 101.6 0)
+			(at 280.67 101.6 0)
 			(effects
 				(font
@@
 		)
 		(property "LCSC#" "C2907113"
-			(at 285.75 101.6 90)
+			(at 280.67 101.6 90)
 			(effects
 				(font
@@
 		)
 		(property "Sim.Device" ""
-			(at 285.75 101.6 0)
+			(at 280.67 101.6 0)
 			(effects
 				(font
@@
 		)
 		(property "Sim.Pins" ""
-			(at 285.75 101.6 0)
+			(at 280.67 101.6 0)
 			(effects
 				(font
@@
 		)
 		(property "Sim.Type" ""
-			(at 285.75 101.6 0)
+			(at 280.67 101.6 0)
 			(effects
 				(font
