File: kicad/mdb-bridge-esp32s3/mdb-bridge-esp32s3.kicad_sch (KiCad schematic)
At the start: 51 parts, among them J1 MDB_Connector, J2 USB_C_Receptacle_USB2.0_16P, J4 Conn_Coaxial, J8 Conn_01x04_Pin, J9 MDB_Connector, Q5 MMBT3906, SW1 SW_Push, U1 TLP785, U17 LM2594HVM-5.0, U2 AP2112K-3.3, U3 ESP32-S3FH4R2, U4 TLP785, Y1 40MHz

Commit message: fix(kicad): optoacopladores com LCSC# C128776 (TLP185 GR) em todos os projetos
C45445 (TLP785 DIP4 SMD) não casa com o footprint SOP-4_3.8x4.1mm.
Troca para C128776 nos esquemáticos de mdb-slave-esp32s3,
mdb-slave-esp32s3-sim7080g e mdb-bridge-esp32s3 (PCBs dos dois
primeiros já estavam corrigidos) e no PCB do mdb-bridge-esp32s3.
Parts:
- U1, U4: LCSC# C45445 -> C128776
Changed lines of the file:
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@@
 			)
 		)
-		(property "LCSC#" "C45445"
+		(property "LCSC#" "C128776"
 			(at 358.14 82.55 0)
 			(effects
@@
 			)
 		)
-		(property "LCSC#" "C45445"
+		(property "LCSC#" "C128776"
 			(at 358.14 97.79 0)
 			(effects

Commit message: fix(kicad): ferrite do VDD3P3 do ESP32 com LCSC# 120R/2A
0603 -> C14709 (Murata BLM18PG121SN1D, 120R@100MHz, 2A, 50mOhm, Basic)
0402 -> C88970 (Murata BLM15PX121SN1D, 120R@100MHz, 2A, 55mOhm)

mini: substitui C14182 (GZ1005D601TF, 100mA, 900mOhm), subdimensionada
para os picos de TX do WiFi.
Parts:
- FB2: LCSC# C304319 -> C14709
Changed lines of the file:
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@@
 			)
 		)
-		(property "LCSC#" "C304319"
+		(property "LCSC#" "C14709"
 			(at 137.16 30.48 90)
 			(effects

Commit message: kicad: unify LCSC codes under LCSC# and add PCBWay production files
- mdb-bridge-esp32s3: move LED1 C5349957 from LCSC Part to LCSC#
- add PCBWay production files (BOM, CPL, IPC netlist, gerbers) for
  mdb-bridge-esp32s3, mdb-slave-esp32s3, mdb-slave-esp32s3-mini and
  mdb-slave-esp32s3-sim7080g
Parts:
- LED1: LCSC Part C5349957 -> (none); LCSC# (none) -> C5349957
Changed lines of the file:
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@@
 			)
 		)
-		(property "LCSC Part" "C5349957"
+		(property "LCSC#" "C5349957"
 			(at 321.31 246.38 0)
 			(effects

Commit message: fix(kicad): MDB TX optocoupler LED resistor 470R -> 100R in all projects
With 470R the TX optocoupler LED only gets ~4.3 mA, so the
phototransistor cannot sink the >= 15 mA @ 1 V the MDB 4.2 spec
requires from a peripheral transmitter. Some VMCs never see our ACK
and keep resending RESET. ngspice: 470R fails even at CTR 300%;
100R sinks ~17 mA at < 0.5 V with CTR >= 100% (TLP185 GR).
GPIO5 current ~17 mA, within the ESP32-S3 default drive strength.

- mdb-slave-esp32s3, -mini, mdb-bridge-esp32s3: R5
- mdb-slave-esp32s3-sim7080g: R18
- LCSC# C22775 (UNI-ROYAL 0603WAF1000T5E) / C25076 for 0402 (mini)
- PCBWay BOM and positions updated; gerbers unchanged

RX resistors (R2 / R16) stay 470R: the spec caps peripheral receive
current at 15 mA @ 4 V.

Refs #76, #77
Parts:
- R5: value 470R -> 100R; LCSC# C114669 -> C22775
Changed lines of the file:
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@@
 			)
 		)
-		(property "Value" "470R"
+		(property "Value" "100R"
 			(at 373.38 105.4099 0)
 			(effects
@@
 			)
 		)
-		(property "LCSC#" "C114669"
+		(property "LCSC#" "C22775"
 			(at 370.84 104.14 0)
 			(effects
