File: kicad/mdb-slave-esp32s3-mini/mdb-slave-esp32s3-mini.kicad_pcb (KiCad board)
At the start: 2 copper layers, 26.6 x 38.7 mm, 43 parts, among them J1 MDB_Connector, J2 USB_C_Receptacle_USB2.0_16P, SW1 SW_Push, U1 TLP785, U3 ESP32-S3FH4R2, U4 TLP785, U5 LM2594HVM-3.3, Y1 40MHz

Commit message: fix(kicad): MDB TX optocoupler LED resistor 470R -> 100R in all projects
With 470R the TX optocoupler LED only gets ~4.3 mA, so the
phototransistor cannot sink the >= 15 mA @ 1 V the MDB 4.2 spec
requires from a peripheral transmitter. Some VMCs never see our ACK
and keep resending RESET. ngspice: 470R fails even at CTR 300%;
100R sinks ~17 mA at < 0.5 V with CTR >= 100% (TLP185 GR).
GPIO5 current ~17 mA, within the ESP32-S3 default drive strength.

- mdb-slave-esp32s3, -mini, mdb-bridge-esp32s3: R5
- mdb-slave-esp32s3-sim7080g: R18
- LCSC# C22775 (UNI-ROYAL 0603WAF1000T5E) / C25076 for 0402 (mini)
- PCBWay BOM and positions updated; gerbers unchanged

RX resistors (R2 / R16) stay 470R: the spec caps peripheral receive
current at 15 mA @ 4 V.

Refs #76, #77
Parts:
- R5: value 470R -> 100R
Changed lines of the file:
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@@
 			)
 		)
-		(property "Value" "470R"
+		(property "Value" "100R"
 			(at 0 1.17 0)
 			(layer "F.Fab")
@@
 			)
 		)
-		(property "LCSC#" "C25117"
+		(property "LCSC#" "C25076"
 			(at 0 0 0)
 			(unlocked yes)
