File: kicad/mdb-slave-esp32s3-mini/mdb-slave-esp32s3-mini.kicad_sch (KiCad schematic)
At the start: 41 parts, among them J1 MDB_Connector, J2 USB_C_Receptacle_USB2.0_16P, SW1 SW_Push, U1 TLP785, U3 ESP32-S3FH4R2, U4 TLP785, U5 LM2594HVM-3.3, Y1 40MHz

Commit message: fix(kicad): corrige LCSC# de SW1, U1 e U4 no mdb-slave-esp32s3-mini
LCSC# não correspondia ao footprint (apontado pela PCBWay):
- SW1: C42435421 (Khon 6x3.5mm, acionamento vertical) -> C388883
  (Panasonic EVQP7C01P, casa com SW_SPST_EVQP7C)
- U1/U4: C45445 (TLP785 DIP4 SMD, 6.5x4.6mm) -> C128776
  (TLP185 GR, SO4 3.7x4.55mm P2.54, casa com SOP-4_3.8x4.1mm;
  mesma peça usada pela PCBWay na montagem)
Parts:
- SW1: LCSC# C42435421 -> C388883
- U1, U4: LCSC# C45445 -> C128776
Changed lines of the file:
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@@
 			)
 		)
-		(property "LCSC#" "C45445"
+		(property "LCSC#" "C128776"
 			(at 358.14 88.9 0)
 			(effects
@@
 			)
 		)
-		(property "LCSC#" "C42435421"
+		(property "LCSC#" "C388883"
 			(at 175.26 115.57 0)
 			(effects
@@
 			)
 		)
-		(property "LCSC#" "C45445"
+		(property "LCSC#" "C128776"
 			(at 358.14 104.14 0)
 			(effects

Commit message: fix(kicad): ferrite do VDD3P3 do ESP32 com LCSC# 120R/2A
0603 -> C14709 (Murata BLM18PG121SN1D, 120R@100MHz, 2A, 50mOhm, Basic)
0402 -> C88970 (Murata BLM15PX121SN1D, 120R@100MHz, 2A, 55mOhm)

mini: substitui C14182 (GZ1005D601TF, 100mA, 900mOhm), subdimensionada
para os picos de TX do WiFi.
Parts:
- FB2: LCSC# C14182 -> C88970
Changed lines of the file:
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@@
 			)
 		)
-		(property "LCSC#" "C14182"
+		(property "LCSC#" "C88970"
 			(at 137.16 30.48 90)
 			(effects

Commit message: fix(kicad): MDB TX optocoupler LED resistor 470R -> 100R in all projects
With 470R the TX optocoupler LED only gets ~4.3 mA, so the
phototransistor cannot sink the >= 15 mA @ 1 V the MDB 4.2 spec
requires from a peripheral transmitter. Some VMCs never see our ACK
and keep resending RESET. ngspice: 470R fails even at CTR 300%;
100R sinks ~17 mA at < 0.5 V with CTR >= 100% (TLP185 GR).
GPIO5 current ~17 mA, within the ESP32-S3 default drive strength.

- mdb-slave-esp32s3, -mini, mdb-bridge-esp32s3: R5
- mdb-slave-esp32s3-sim7080g: R18
- LCSC# C22775 (UNI-ROYAL 0603WAF1000T5E) / C25076 for 0402 (mini)
- PCBWay BOM and positions updated; gerbers unchanged

RX resistors (R2 / R16) stay 470R: the spec caps peripheral receive
current at 15 mA @ 4 V.

Refs #76, #77
Parts:
- R5: value 470R -> 100R; LCSC# C25117 -> C25076
Changed lines of the file:
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@@
 			)
 		)
-		(property "Value" "470R"
+		(property "Value" "100R"
 			(at 373.38 111.7599 0)
 			(effects
@@
 			)
 		)
-		(property "LCSC#" "C25117"
+		(property "LCSC#" "C25076"
 			(at 370.84 110.49 0)
 			(effects

Commit message: refactor(kicad): move 3D models to easyeda2kicad layout and sync PCBs
- replace per-project 3d-models/ with kicad-libs/<MPN>.3dshapes using
  EasyEDA models fetched by LCSC#, aligned to the KiCad footprints:
  GT-USB-7010ASV, DLL-5566-6A, SLH0704S101MTT, SIM7080G,
  SF72S006VBDR2500 (wrl) and 479480001 (mini antenna)
- buzzer and WS2812B-2020 keep the previous models (no usable EasyEDA one)
- mdb-bridge L6 now has a 3D model
- sim7080g: SIM7080G symbol/footprint moved to kicad-libs with
  project fp-lib-table and sym-lib-table
- mini: AE1 LCSC# C152351
- slave and sim7080g: PCB Value fields synced with the schematic
- re-rendered board PNGs
Parts:
- AE1: LCSC# (none) -> C152351
Changed lines of the file:
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@@
+			)
+		)
+		(property "LCSC#" "C152351"
+			(at 29.21 99.06 0)
+			(effects
+				(font
+					(size 1.27 1.27)
+				)
+				(hide yes)
 			)
 		)
